File: LedWall.kicad_pcb (KiCad board)
At the start: 2 copper layers, 205 x 205 mm, 63 parts, among them J1 Conn_02x05_Odd_Even, J2 Conn_02x05_Odd_Even, J3 Conn_02x05_Odd_Even, J4 Conn_02x05_Odd_Even, U2 TPS5430DDA

Commit message: Updated project to kicad 6 and changed PCB
Parts:
- removed U2: TPS5430DDA, Package_SO:TI_SO-PowerPAD-8_ThermalVias
- added C29: 100n/10V, Capacitor_SMD:C_0603_1608Metric_Pad1.08x0.95mm_HandSolder, F.Cu at (211.1, 54.4)
- added D27: B340, Diode_SMD:D_SOD-123, F.Cu at (174.8, 74.7)
- added H1: ToolingHole, JLC:JLC_toolinghole, F.Cu at (49.8, 41.4)
- added H2: ToolingHole, JLC:JLC_toolinghole, F.Cu at (235.1, 243.8)
- added R4: 10k, Resistor_SMD:R_0603_1608Metric_Pad0.98x0.95mm_HandSolder, F.Cu at (210.1, 51.8)
- added R5: 7k5, Resistor_SMD:R_0603_1608Metric_Pad0.98x0.95mm_HandSolder, F.Cu at (173.6, 89.5)
- added R6: 20k, Resistor_SMD:R_0603_1608Metric_Pad0.98x0.95mm_HandSolder, F.Cu at (209.0, 54.4)
- added TP1: TestPoint, TestPoint:TestPoint_Loop_D1.80mm_Drill1.0mm_Beaded, F.Cu at (49.2, 63.6)
- added TP2: TestPoint, TestPoint:TestPoint_Loop_D1.80mm_Drill1.0mm_Beaded, F.Cu at (232.2, 80.9)
- added TP3: TestPoint, TestPoint:TestPoint_Loop_D1.80mm_Drill1.0mm_Beaded, F.Cu at (56.6, 121.4)
- added TP4: TestPoint, TestPoint:TestPoint_Loop_D1.80mm_Drill1.0mm_Beaded, F.Cu at (232.2, 161.9)
- added TP5: TestPoint, TestPoint:TestPoint_Loop_D1.80mm_Drill1.0mm_Beaded, F.Cu at (59.4, 202.6)
- added TP6: TestPoint, TestPoint:TestPoint_Loop_D1.80mm_Drill1.0mm_Beaded, F.Cu at (49.8, 234.2)
- added TP7: TestPoint, TestPoint:TestPoint_Loop_D1.80mm_Drill1.0mm_Beaded, F.Cu at (181.1, 77.4)
- added TP8: TestPoint, TestPoint:TestPoint_Loop_D1.80mm_Drill1.0mm_Beaded, F.Cu at (77.2, 95.5)
- added TP9: TestPoint, TestPoint:TestPoint_Loop_D1.80mm_Drill1.0mm_Beaded, F.Cu at (206.2, 52.3)
- added U1: TPS5430DDA, Package_SO:TI_SO-PowerPAD-8_ThermalVias, F.Cu at (175.0, 83.8)
- C1, C10, C11, C12, C13, C14, C15, C16, C17, C18, C19, C2, C20, C21, C22, C23, C24, C25, C3, C4, C5, C6, C7, C8, C9: value 100n -> 100n/10V
- C27: value 220u -> 10u/50V; footprint Capacitor_SMD:CP_Elec_6.3x5.4 -> Capacitor_SMD:C_1206_3216Metric_Pad1.33x1.80mm_HandSolder
- D26: footprint Diode_SMD:D_SMC -> Diode_SMD:D_SOD-123
- L1: value 22u -> 650u; footprint Inductor_SMD:L_Taiyo-Yuden_MD-4040 -> Inductor_SMD:L_Bourns_SRR1208_12.7x12.7mm
- R2: value 10k -> 20k
- R3: value 3.24k -> 20k
- moved R2 145.3 mm to (54.9, 64.5), turned to -90 degrees
- moved L1 45.0 mm to (162.8, 80.4)
- moved R3 42.6 mm to (171.8, 88.0)
- moved C26 41.6 mm to (170.2, 79.4)
- moved C28 41.6 mm to (181.0, 83.3)
- moved C27 41.2 mm to (170.9, 91.9), turned to 180 degrees
- moved D26 40.3 mm to (185.2, 82.1), turned to 0 degrees
- moved C23 13.2 mm to (144.2, 228.2), turned to 180 degrees
- moved C24 11.9 mm to (185.3, 228.2), turned to 180 degrees
- moved C20 11.8 mm to (222.9, 179.8)
- moved C25 11.3 mm to (226.2, 228.2), turned to 180 degrees
- moved C19 11.2 mm to (182.0, 179.8)
- moved C18 10.7 mm to (140.8, 179.8)
- moved C17 10.2 mm to (99.9, 179.8)
- moved C7 10.2 mm to (99.7, 97.8)
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Connections:
- C26 pad 1: Net-(C26-Pad1) -> /Led Wall Power/PH
- C26 pad 2: Net-(C26-Pad2) -> /Led Wall Power/BOOT
- C27 pad 1: +5V -> GND
- C27 pad 2: GND -> +5V
- C28 pad 2: VDC -> /Led Wall Power/VDC+
- D1 pad 4: Net-(D1-Pad4) -> /DataInFiltered
- D26 pad 1: Net-(C26-Pad1) -> /Led Wall Power/VDC+
- D26 pad 2: GND -> VDC
- L1 pad 1: Net-(C26-Pad1) -> /Led Wall Power/PH
- R1 pad 1: Net-(D1-Pad4) -> /DataInFiltered
- R2 pad 1: +5V -> /DataInFiltered
- R2 pad 2: Net-(R2-Pad2) -> GND
- R3 pad 1: Net-(R2-Pad2) -> +5V
- R3 pad 2: GND -> /Led Wall Power/VSENSE
Routing:
- net +5V: track 9.83 -> 1163.7 mm
- net /Led Wall Power/EN: track 0.00 -> 81.0 mm, vias 0 -> 1
- net Net-(D4-Pad2): track 0.00 -> 37.4 mm
- net /DataInFiltered: track 0.00 -> 10.6 mm
- net /PWR_EN: track 237.8 -> 228.6 mm, vias 3 -> 1
- net Net-(R2-Pad2): track 4.56 -> 0.00 mm
- net /Led Wall Power/VSENSE: track 0.00 -> 3.91 mm
- net /DataOut: track 197.9 -> 201.7 mm
- net Net-(D15-Pad2): track 43.3 -> 47.0 mm
- net Net-(D1-Pad4): track 3.27 -> 0.00 mm
- net Net-(D10-Pad4): track 42.8 -> 46.0 mm
- net Net-(C26-Pad2): track 2.88 -> 0.00 mm
- net /Led Wall Power/BOOT: track 0.00 -> 2.61 mm
- net /DataIn: track 22.4 -> 23.8 mm
- net Net-(D11-Pad4): track 42.9 -> 44.1 mm
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- added copper zone on F.Cu, net /Led Wall Power/PH
- added copper zone on F.Cu, net /Led Wall Power/VDC+
- removed copper zone on F.Cu, net Net-(C26-Pad1)
Other:
- net class Default removed
- board text added: "JLCJLCJLCJLC"
- board text added: "LedWall rev1 2022-07-21"
- board text added: "Vin: 12V-36V"

Commit message: Change DC/DC components and split schematic
Parts:
- added C30: 100n/10V, Capacitor_SMD:C_0603_1608Metric_Pad1.08x0.95mm_HandSolder, F.Cu at (211.1, 54.4)
- C27: value 10u/50V -> 150u/50V; footprint Capacitor_SMD:C_1206_3216Metric_Pad1.33x1.80mm_HandSolder -> Capacitor_SMD:C_Elec_10x10.2
- C29: value 100n/10V -> 10u/50V; footprint Capacitor_SMD:C_0603_1608Metric_Pad1.08x0.95mm_HandSolder -> Capacitor_SMD:C_1206_3216Metric_Pad1.33x1.80mm_HandSolder
- L1: value 650u -> 47u; footprint Inductor_SMD:L_Bourns_SRR1208_12.7x12.7mm -> Ledwall:YNR6045-470M
- R1: value 22 -> 270R
- R2: value 20k -> 22
- moved C29 38.7 mm to (178.6, 75.4), turned to 90 degrees
- moved TP7 23.2 mm to (161.2, 65.7)
- moved C28 9.24 mm to (176.2, 75.4)
- moved D27 9.24 mm to (170.0, 66.9)
- moved C26 9.24 mm to (165.4, 71.6)
- moved R5 9.24 mm to (168.8, 81.7)
- moved R3 9.24 mm to (167.0, 80.1)
- moved U1 9.24 mm to (170.2, 76.0)
- moved L1 8.67 mm to (161.2, 71.8), turned to 0 degrees
- moved D26 8.52 mm to (182.2, 74.2)
- moved C27 6.08 mm to (166.2, 88.0)
- moved R2 2.70 mm to (54.0, 62.0), turned to 180 degrees
- moved R1 2.59 mm to (54.9, 64.4), turned to 90 degrees
- moved H2 2.03 mm to (233.0, 243.8)
Connections:
- net /Led Wall Power/BOOT renamed /Power/BOOT
- net /Led Wall Power/PH renamed /Power/PH
- net /Led Wall Power/VSENSE renamed /Power/VSENSE
- C28 pad 2: /Led Wall Power/VDC+ -> /Power/VDC+
- C29 pad 1: /Led Wall Power/EN -> GND
- C29 pad 2: GND -> /Power/VDC+
- D1 pad 4: /DataInFiltered -> /LEDs/DataInFiltered
- D26 pad 1: /Led Wall Power/VDC+ -> /Power/VDC+
- R1 pad 1: /DataInFiltered -> +5V
- R1 pad 2: /DataIn -> /LEDs/DataInFiltered
- R2 pad 1: /DataInFiltered -> /LEDs/DataInFiltered
- R2 pad 2: GND -> /DataIn
- R4 pad 2: /Led Wall Power/EN -> /Power/EN
- R6 pad 1: /Led Wall Power/EN -> /Power/EN
- TP1 pad 1: /DataInFiltered -> /LEDs/DataInFiltered
- TP9 pad 1: /Led Wall Power/EN -> /Power/EN
- U1 pad 5: /Led Wall Power/EN -> /Power/EN
- U1 pad 7: /Led Wall Power/VDC+ -> /Power/VDC+
Routing:
- net /Power/EN: track 0.00 -> 93.4 mm, vias 0 -> 1
- net /Led Wall Power/EN: track 81.0 -> 0.00 mm, vias 1 -> 0
- net +5V: track 1163.7 -> 1190.2 mm
- net /LEDs/DataInFiltered: track 0.00 -> 10.6 mm
- net /DataInFiltered: track 10.6 -> 0.00 mm
- net VDC: vias 28 -> 53
- net GND: vias 5020 -> 5018
- added copper zone on F.Cu, net /Power/VDC+
- removed copper zone on F.Cu, net /Led Wall Power/VDC+

Commit message: Change LED to one in JLC stock
Parts:
- moved TP7 1.70 mm to (159.6, 66.4)
Routing:
- net GND: vias 5018 -> 5026
Other:
- board text added: "Skrooter Audio"
Changed lines of the file:
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@@
   )
   (footprint "TestPoint:TestPoint_Loop_D1.80mm_Drill1.0mm_Beaded" (layer "F.Cu")
-    (at 161.163 65.659)
+    (at 159.639 66.421)
     (descr "wire loop with bead as test point, loop diameter 1.8mm, hole diameter 1.0mm")
     (tags "test point wire loop bead")
@@
     (effects (font (size 1 1) (thickness 0.15)) (justify mirror))
   )
+  (gr_text "Skrooter Audio" (at 183.007 241.808) (layer "F.SilkS")
+    (effects (font (size 3 3) (thickness 0.5)))
+  )
   (gr_text "LedWall rev1\n2022-07-21" (at 213.614 241.808) (layer "F.SilkS")
     (effects (font (size 1.5 1.5) (thickness 0.3)))
@@
   (segment (start 106.772 61.722) (end 103.95 58.9) (width 0.25) (layer "F.Cu") (net 2))
   (segment (start 139.672 61.722) (end 106.772 61.722) (width 0.25) (layer "F.Cu") (net 2))
-  (segment (start 147.645 61.595) (end 144.95 58.9) (width 0.25) (layer "F.Cu") (net 3))
-  (segment (start 180.545 61.595) (end 147.645 61.595) (width 0.25) (layer "F.Cu") (net 3))
-  (segment (start 181.05 62.1) (end 180.545 61.595) (width 0.25) (layer "F.Cu") (net 3))
+  (segment (start 181.05 62.1) (end 177.85 58.9) (width 0.25) (layer "F.Cu") (net 3))
+  (segment (start 177.85 58.9) (end 144.95 58.9) (width 0.25) (layer "F.Cu") (net 3))
   (segment (start 200.533 61.341) (end 198.092 58.9) (width 0.25) (layer "F.Cu") (net 4))
   (segment (start 222.05 62.1) (end 221.291 61.341) (width 0.25) (layer "F.Cu") (net 4))
@@
   (via (at 50.482619 118.665) (size 0.8) (drill 0.4) (layers "F.Cu" "B.Cu") (free) (net 13))
   (via (at 218.122619 116.125) (size 0.8) (drill 0.4) (layers "F.Cu" "B.Cu") (free) (net 13))
+  (via (at 157.162619 62.785) (size 0.8) (drill 0.4) (layers "F.Cu" "B.Cu") (free) (net 13))
   (via (at 93.662619 75.485) (size 0.8) (drill 0.4) (layers "F.Cu" "B.Cu") (free) (net 13))
   (via (at 154.622619 111.045) (size 0.8) (drill 0.4) (layers "F.Cu" "B.Cu") (free) (net 13))
@@
   (via (at 131.762619 138.985) (size 0.8) (drill 0.4) (layers "F.Cu" "B.Cu") (free) (net 13))
   (via (at 88.582619 205.025) (size 0.8) (drill 0.4) (layers "F.Cu" "B.Cu") (free) (net 13))
+  (via (at 162.242619 62.785) (size 0.8) (drill 0.4) (layers "F.Cu" "B.Cu") (free) (net 13))
   (via (at 96.202619 72.945) (size 0.8) (drill 0.4) (layers "F.Cu" "B.Cu") (free) (net 13))
   (via (at 205.422619 205.025) (size 0.8) (drill 0.4) (layers "F.Cu" "B.Cu") (free) (net 13))
@@
   (via (at 58.102619 78.025) (size 0.8) (drill 0.4) (layers "F.Cu" "B.Cu") (free) (net 13))
   (via (at 139.382619 172.005) (size 0.8) (drill 0.4) (layers "F.Cu" "B.Cu") (free) (net 13))
+  (via (at 164.782619 62.785) (size 0.8) (drill 0.4) (layers "F.Cu" "B.Cu") (free) (net 13))
   (via (at 75.882619 161.845) (size 0.8) (drill 0.4) (layers "F.Cu" "B.Cu") (free) (net 13))
   (via (at 152.082619 184.705) (size 0.8) (drill 0.4) (layers "F.Cu" "B.Cu") (free) (net 13))
@@
   (via (at 126.682619 133.905) (size 0.8) (drill 0.4) (layers "F.Cu" "B.Cu") (free) (net 13))
   (via (at 93.662619 133.905) (size 0.8) (drill 0.4) (layers "F.Cu" "B.Cu") (free) (net 13))
+  (via (at 147.002619 60.245) (size 0.8) (drill 0.4) (layers "F.Cu" "B.Cu") (free) (net 13))
   (via (at 116.522619 235.505) (size 0.8) (drill 0.4) (layers "F.Cu" "B.Cu") (free) (net 13))
   (via (at 185.102619 199.945) (size 0.8) (drill 0.4) (layers "F.Cu" "B.Cu") (free) (net 13))
@@
   (via (at 50.482619 144.065) (size 0.8) (drill 0.4) (layers "F.Cu" "B.Cu") (free) (net 13))
   (via (at 91.122619 156.765) (size 0.8) (drill 0.4) (layers "F.Cu" "B.Cu") (free) (net 13))
+  (via (at 167.322619 62.785) (size 0.8) (drill 0.4) (layers "F.Cu" "B.Cu") (free) (net 13))
   (via (at 91.122619 57.705) (size 0.8) (drill 0.4) (layers "F.Cu" "B.Cu") (free) (net 13))
   (via (at 147.002619 118.665) (size 0.8) (drill 0.4) (layers "F.Cu" "B.Cu") (free) (net 13))
@@
   (via (at 225.742619 205.025) (size 0.8) (drill 0.4) (layers "F.Cu" "B.Cu") (free) (net 13))
   (via (at 169.862619 238.045) (size 0.8) (drill 0.4) (layers "F.Cu" "B.Cu") (free) (net 13))
+  (via (at 169.862619 62.785) (size 0.8) (drill 0.4) (layers "F.Cu" "B.Cu") (free) (net 13))
   (via (at 111.442619 166.925) (size 0.8) (drill 0.4) (layers "F.Cu" "B.Cu") (free) (net 13))
   (via (at 129.222619 205.025) (size 0.8) (drill 0.4) (layers "F.Cu" "B.Cu") (free) (net 13))
@@
   (via (at 147.002619 47.545) (size 0.8) (drill 0.4) (layers "F.Cu" "B.Cu") (free) (net 13))
   (via (at 42.862619 121.205) (size 0.8) (drill 0.4) (layers "F.Cu" "B.Cu") (free) (net 13))
+  (via (at 172.402619 62.785) (size 0.8) (drill 0.4) (layers "F.Cu" "B.Cu") (free) (net 13))
   (via (at 225.742619 50.085) (size 0.8) (drill 0.4) (layers "F.Cu" "B.Cu") (free) (net 13))
   (via (at 131.762619 202.485) (size 0.8) (drill 0.4) (layers "F.Cu" "B.Cu") (free) (net 13))
@@
   (via (at 164.782619 161.845) (size 0.8) (drill 0.4) (layers "F.Cu" "B.Cu") (free) (net 13))
   (via (at 202.882619 83.105) (size 0.8) (drill 0.4) (layers "F.Cu" "B.Cu") (free) (net 13))
+  (via (at 159.702619 62.785) (size 0.8) (drill 0.4) (layers "F.Cu" "B.Cu") (free) (net 13))
   (via (at 93.662619 78.025) (size 0.8) (drill 0.4) (layers "F.Cu" "B.Cu") (free) (net 13))
   (via (at 111.442619 151.685) (size 0.8) (drill 0.4) (layers "F.Cu" "B.Cu") (free) (net 13))
@@
         (xy 166.165 71.4536)
         (xy 157.498 71.4536)
-        (xy 157.498 63.6206)
-        (xy 174.196 63.6206)
+        (xy 157.498 64.3826)
+        (xy 174.196 64.3826)
       )
     )
@@
       03e3bdf5-efcb-4ca2-bb81-cce04c8f884b
       03fa257f-44c1-4a8f-b311-a36690d55a0a
+      03fe72de-ec81-4da8-88c5-05feae4f971a
       0404cea0-796b-4ca3-9480-98d80f2d81df
       040679c1-8c3d-45c0-b910-7d6746b25bbf
@@
       33b5ccd5-8952-46a0-a50f-d37b752bf442
       33b84fff-60cd-4d03-aa84-36a36706e7ed
+      33bd784a-d0dc-4c35-b403-0a08e2a1bbc6
       33c69f9d-bd23-4bf5-8d29-591374bca576
       33cce9ca-0c02-44f9-a4a1-cdd099438e33
@@
       3dd954d6-abff-40d3-81db-61b25bdff078
       3ddf41b2-c032-4dc5-b336-e9a56580106b
+      3de77b6a-ee62-4ff0-90f6-31934b51eaea
       3df3c5bb-5571-4154-9824-c7d2d2117a73
       3e0c5c08-0d54-4c28-af71-77b3c31d1315
@@
       5d45aeb0-49cc-43c7-9a75-ef96fec61976
       5d5c39b0-b623-4a20-bf7d-b8175c9fcf4c
+      5d65c0f8-8121-4e17-b2f0-a682aa8d32ae
       5d6d1a24-3fae-481f-bf36-896fdde55679
       5d7baf13-136f-43a9-b725-ea899beefe6b
@@
       972b0d7c-8b65-4e9a-94eb-700225a61630
       9735b16e-87ba-4dd7-9f8b-0c7c7635da18
+      9736113b-17a9-4861-8a22-037fb1eb6aea
       97422557-ba5c-4f63-8e74-7a77513d017d
       974cb764-7852-41f0-a462-c5af71e299b9
@@
       a53a2136-4d70-446a-b690-c6d17e9733e1
       a541ea01-d386-4be5-af82-6024c9c8a063
+      a54af14f-7da0-49a9-a89d-c263861882cc
       a54f3212-2659-4eaf-9049-6ad2bb530bc3
       a568cef2-3e9c-43cd-b90c-fdb1fbcdc774
@@
       f7b3d8b5-b2fa-460a-a72b-129592c9eced
       f7bed1e7-c580-43de-977d-54f85e089f99
+      f7c1240c-a300-4568-bb1f-a22b275dc355
       f81e30d1-e39f-4fa9-a189-72fdf7d47131
       f8207119-e174-4a5c-af40-3fac329e62e0
@@
       fa07b115-f600-43b4-a9f7-6f65611580f6
       fa0926cf-2c56-4c84-843d-6b2f903153ad
+      fa0c4ad2-70da-4bf0-a58e-270f3fba1444
       fa161a59-67a5-4c69-8e61-b9f521f2643c
       fa229fd4-7154-4162-aac1-aee73629218d
