File: LedWall.kicad_pcb (KiCad board)
At the start: 2 copper layers, 205 x 205 mm, 85 parts, among them J101 Conn_02x05_Odd_Even, J102 Conn_02x05_Odd_Even, J103 Conn_02x05_Odd_Even, J104 Conn_02x05_Odd_Even, U201 TPS5430DDA

Commit message: Add GND testpoints
Each other testpoint now has its own ground reference

fix #6
Parts:
- added TP204: TestPoint, TestPoint:TestPoint_Loop_D1.80mm_Drill1.0mm_Beaded, F.Cu at (202.2, 52.3)
- added TP205: TestPoint, TestPoint:TestPoint_Loop_D1.80mm_Drill1.0mm_Beaded, F.Cu at (154.9, 66.4)
- added TP206: TestPoint, TestPoint:TestPoint_Loop_D1.80mm_Drill1.0mm_Beaded, F.Cu at (151.9, 84.3)
- added TP212: TestPoint, TestPoint:TestPoint_Loop_D1.80mm_Drill1.0mm_Beaded, F.Cu at (223.5, 236.7)
- added TP213: TestPoint, TestPoint:TestPoint_Loop_D1.80mm_Drill1.0mm_Beaded, F.Cu at (221.0, 173.2)
- added TP214: TestPoint, TestPoint:TestPoint_Loop_D1.80mm_Drill1.0mm_Beaded, F.Cu at (143.8, 71.6)
- added TP215: TestPoint, TestPoint:TestPoint_Loop_D1.80mm_Drill1.0mm_Beaded, F.Cu at (209.3, 69.1)
- added TP216: TestPoint, TestPoint:TestPoint_Loop_D1.80mm_Drill1.0mm_Beaded, F.Cu at (227.1, 152.9)
- added TP307: TestPoint, TestPoint:TestPoint_Loop_D1.80mm_Drill1.0mm_Beaded, F.Cu at (49.3, 59.4)
- added TP308: TestPoint, TestPoint:TestPoint_Loop_D1.80mm_Drill1.0mm_Beaded, F.Cu at (236.2, 80.8)
- added TP309: TestPoint, TestPoint:TestPoint_Loop_D1.80mm_Drill1.0mm_Beaded, F.Cu at (60.5, 121.4)
- added TP310: TestPoint, TestPoint:TestPoint_Loop_D1.80mm_Drill1.0mm_Beaded, F.Cu at (228.1, 162.1)
- added TP311: TestPoint, TestPoint:TestPoint_Loop_D1.80mm_Drill1.0mm_Beaded, F.Cu at (63.5, 202.7)
- added TP312: TestPoint, TestPoint:TestPoint_Loop_D1.80mm_Drill1.0mm_Beaded, F.Cu at (52.8, 236.7)
- moved TP208 0.25 mm to (221.0, 177.0)
- moved TP209 0.25 mm to (143.8, 67.8)
- moved TP305 0.13 mm to (59.4, 202.7)
- moved TP302 0.13 mm to (232.2, 80.8)
- renumbered TP204 to TP207, TP205 to TP208, TP206 to TP209, TP207 to TP210, TP208 to TP211
Routing:
- net GND: vias 5070 -> 5039

Commit message: Add 12V testpoint
fix #3
Parts:
- added TP201: TestPoint, TestPoint:TestPoint_Loop_D1.80mm_Drill1.0mm_Beaded, F.Cu at (159.5, 44.2)
- added TP205: TestPoint, TestPoint:TestPoint_Loop_D1.80mm_Drill1.0mm_Beaded, F.Cu at (159.5, 48.8)
- renumbered TP201 to TP202, TP202 to TP203, TP203 to TP204, TP204 to TP206, TP205 to TP207, TP206 to TP208, TP207 to TP209, TP208 to TP210, TP209 to TP211, TP210 to TP212, TP211 to TP213, TP212 to TP214, TP213 to TP215, TP214 to TP216, TP215 to TP217, TP216 to TP218
Routing:
- net GND: vias 5039 -> 5037
Changed lines of the file:
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@@
     (property "Sheetname" "Power")
     (attr through_hole)
-    (fp_text reference "TP204" (at 0.7 2.5) (layer "F.SilkS")
+    (fp_text reference "TP206" (at 0.7 2.5) (layer "F.SilkS")
       (effects (font (size 1 1) (thickness 0.15)))
     )
@@
     (property "Sheetname" "Power")
     (attr through_hole)
-    (fp_text reference "TP215" (at 4.064 0) (layer "F.SilkS")
+    (fp_text reference "TP217" (at 4.064 0) (layer "F.SilkS")
       (effects (font (size 1 1) (thickness 0.15)))
     )
@@
     (property "Sheetname" "Power")
     (attr through_hole)
-    (fp_text reference "TP202" (at 4.191 0.127) (layer "F.SilkS")
+    (fp_text reference "TP203" (at 4.191 0.127) (layer "F.SilkS")
       (effects (font (size 1 1) (thickness 0.15)))
     )
@@
     (property "Sheetname" "Power")
     (attr through_hole)
-    (fp_text reference "TP203" (at 0.4572 -3.4544) (layer "F.SilkS")
+    (fp_text reference "TP204" (at 0.4572 -3.4544) (layer "F.SilkS")
       (effects (font (size 1 1) (thickness 0.15)))
     )
@@
     (property "Sheetname" "Power")
     (attr through_hole)
-    (fp_text reference "TP214" (at 0.7 2.5) (layer "F.SilkS")
+    (fp_text reference "TP216" (at 0.7 2.5) (layer "F.SilkS")
       (effects (font (size 1 1) (thickness 0.15)))
     )
@@
     (property "Sheetname" "Power")
     (attr through_hole)
-    (fp_text reference "TP201" (at 4.445 -0.889) (layer "F.SilkS")
+    (fp_text reference "TP202" (at 4.445 -0.889) (layer "F.SilkS")
       (effects (font (size 1 1) (thickness 0.15)))
     )
@@
     (property "Sheetname" "Power")
     (attr through_hole)
-    (fp_text reference "TP209" (at -4.064 0) (layer "F.SilkS")
+    (fp_text reference "TP211" (at -4.064 0) (layer "F.SilkS")
       (effects (font (size 1 1) (thickness 0.15)))
     )
@@
   )
   (footprint "TestPoint:TestPoint_Loop_D1.80mm_Drill1.0mm_Beaded" (layer "F.Cu")
+    (at 159.512 48.768)
+    (descr "wire loop with bead as test point, loop diameter 1.8mm, hole diameter 1.0mm")
+    (tags "test point wire loop bead")
+    (property "LCSC" "C238122")
+    (property "Sheetfile" "File: LedWallPower.kicad_sch")
+    (property "Sheetname" "Power")
+    (attr through_hole)
+    (fp_text reference "TP205" (at 4.064 0) (layer "F.SilkS")
+      (effects (font (size 1 1) (thickness 0.15)))
+    )
+    (fp_text value "TestPoint" (at 0 -2.8) (layer "F.Fab")
+      (effects (font (size 1 1) (thickness 0.15)))
+    )
+    (fp_text user "${REFERENCE}" (at 0.7 2.5) (layer "F.Fab")
+      (effects (font (size 1 1) (thickness 0.15)))
+    )
+    (fp_circle (center 0 0) (end 1.5 0) (layer "F.SilkS") (width 0.12) (fill none))
+    (fp_circle (center 0 0) (end 1.8 0) (layer "F.CrtYd") (width 0.05) (fill none))
+    (fp_line (start 0.9 -0.2) (end 0.9 0.2) (layer "F.Fab") (width 0.12))
+    (fp_line (start 0.9 0.2) (end -0.9 0.2) (layer "F.Fab") (width 0.12))
+    (fp_line (start -0.9 -0.2) (end 0.9 -0.2) (layer "F.Fab") (width 0.12))
+    (fp_line (start -0.9 0.2) (end -0.9 -0.2) (layer "F.Fab") (width 0.12))
+    (fp_circle (center 0 0) (end 1.3 0) (layer "F.Fab") (width 0.12) (fill none))
+    (pad "1" thru_hole circle (at 0 0) (size 2 2) (drill 1) (layers *.Cu *.Mask)
+      (net 13 "GND") (pinfunction "1") (pintype "passive"))
+    (model "${KICAD6_3DMODEL_DIR}/TestPoint.3dshapes/TestPoint_Loop_D1.80mm_Drill1.0mm_Beaded.wrl"
+      (offset (xyz 0 0 0))
+      (scale (xyz 1 1 1))
+      (rotate (xyz 0 0 0))
+    )
+  )
+  (footprint "TestPoint:TestPoint_Loop_D1.80mm_Drill1.0mm_Beaded" (layer "F.Cu")
     (at 154.94 66.421)
     (descr "wire loop with bead as test point, loop diameter 1.8mm, hole diameter 1.0mm")
@@
     (property "Sheetname" "Power")
     (attr through_hole)
-    (fp_text reference "TP205" (at 0.7 2.5) (layer "F.SilkS")
+    (fp_text reference "TP207" (at 0.7 2.5) (layer "F.SilkS")
       (effects (font (size 1 1) (thickness 0.15)))
     )
@@
     (property "Sheetname" "Power")
     (attr through_hole)
-    (fp_text reference "TP213" (at 4.064 0) (layer "F.SilkS")
+    (fp_text reference "TP215" (at 4.064 0) (layer "F.SilkS")
       (effects (font (size 1 1) (thickness 0.15)))
     )
@@
     (property "Sheetname" "Power")
     (attr through_hole)
-    (fp_text reference "TP216" (at -4.064 0) (layer "F.SilkS")
+    (fp_text reference "TP218" (at -4.064 0) (layer "F.SilkS")
       (effects (font (size 1 1) (thickness 0.15)))
     )
@@
     (property "Sheetname" "Power")
     (attr through_hole)
-    (fp_text reference "TP208" (at -3.81 0) (layer "F.SilkS")
+    (fp_text reference "TP210" (at -3.81 0) (layer "F.SilkS")
       (effects (font (size 1 1) (thickness 0.15)))
     )
@@
     (property "Sheetname" "Power")
     (attr through_hole)
-    (fp_text reference "TP211" (at -4.064 1.016) (layer "F.SilkS")
+    (fp_text reference "TP213" (at -4.064 1.016) (layer "F.SilkS")
       (effects (font (size 1 1) (thickness 0.15)))
     )
@@
     (property "Sheetname" "Power")
     (attr through_hole)
-    (fp_text reference "TP210" (at 4.064 -0.127) (layer "F.SilkS")
+    (fp_text reference "TP212" (at 4.064 -0.127) (layer "F.SilkS")
       (effects (font (size 1 1) (thickness 0.15)))
     )
@@
     (property "Sheetname" "Power")
     (attr through_hole)
-    (fp_text reference "TP207" (at 0.7 2.5) (layer "F.SilkS")
+    (fp_text reference "TP209" (at 0.7 2.5) (layer "F.SilkS")
       (effects (font (size 1 1) (thickness 0.15)))
     )
@@
     (property "Sheetname" "Power")
     (attr through_hole)
-    (fp_text reference "TP212" (at 0.7 2.5) (layer "F.SilkS")
+    (fp_text reference "TP214" (at 0.7 2.5) (layer "F.SilkS")
       (effects (font (size 1 1) (thickness 0.15)))
     )
@@
   )
   (footprint "TestPoint:TestPoint_Loop_D1.80mm_Drill1.0mm_Beaded" (layer "F.Cu")
+    (at 159.512 44.196)
+    (descr "wire loop with bead as test point, loop diameter 1.8mm, hole diameter 1.0mm")
+    (tags "test point wire loop bead")
+    (property "LCSC" "C238122")
+    (property "Sheetfile" "File: LedWallPower.kicad_sch")
+    (property "Sheetname" "Power")
+    (attr through_hole)
+    (fp_text reference "TP201" (at 4.064 0) (layer "F.SilkS")
+      (effects (font (size 1 1) (thickness 0.15)))
+    )
+    (fp_text value "TestPoint" (at 0 -2.8) (layer "F.Fab")
+      (effects (font (size 1 1) (thickness 0.15)))
+    )
+    (fp_text user "${REFERENCE}" (at 0.7 2.5) (layer "F.Fab")
+      (effects (font (size 1 1) (thickness 0.15)))
+    )
+    (fp_circle (center 0 0) (end 1.5 0) (layer "F.SilkS") (width 0.12) (fill none))
+    (fp_circle (center 0 0) (end 1.8 0) (layer "F.CrtYd") (width 0.05) (fill none))
+    (fp_line (start -0.9 0.2) (end -0.9 -0.2) (layer "F.Fab") (width 0.12))
+    (fp_line (start 0.9 0.2) (end -0.9 0.2) (layer "F.Fab") (width 0.12))
+    (fp_line (start 0.9 -0.2) (end 0.9 0.2) (layer "F.Fab") (width 0.12))
+    (fp_line (start -0.9 -0.2) (end 0.9 -0.2) (layer "F.Fab") (width 0.12))
+    (fp_circle (center 0 0) (end 1.3 0) (layer "F.Fab") (width 0.12) (fill none))
+    (pad "1" thru_hole circle (at 0 0) (size 2 2) (drill 1) (layers *.Cu *.Mask)
+      (net 19 "VDC") (pinfunction "1") (pintype "passive"))
+    (model "${KICAD6_3DMODEL_DIR}/TestPoint.3dshapes/TestPoint_Loop_D1.80mm_Drill1.0mm_Beaded.wrl"
+      (offset (xyz 0 0 0))
+      (scale (xyz 1 1 1))
+      (rotate (xyz 0 0 0))
+    )
+  )
+  (footprint "TestPoint:TestPoint_Loop_D1.80mm_Drill1.0mm_Beaded" (layer "F.Cu")
     (at 151.892 84.328)
     (descr "wire loop with bead as test point, loop diameter 1.8mm, hole diameter 1.0mm")
@@
     (property "Sheetname" "Power")
     (attr through_hole)
-    (fp_text reference "TP206" (at -4.064 0) (layer "F.SilkS")
+    (fp_text reference "TP208" (at -4.064 0) (layer "F.SilkS")
       (effects (font (size 1 1) (thickness 0.15)))
     )
@@
   (via (at 131.762619 207.565) (size 0.8) (drill 0.4) (layers "F.Cu" "B.Cu") (free) (net 13))
   (via (at 119.062619 60.245) (size 0.8) (drill 0.4) (layers "F.Cu" "B.Cu") (free) (net 13))
-  (via (at 159.702619 50.085) (size 0.8) (drill 0.4) (layers "F.Cu" "B.Cu") (free) (net 13))
   (via (at 108.902619 111.045) (size 0.8) (drill 0.4) (layers "F.Cu" "B.Cu") (free) (net 13))
   (via (at 144.462619 169.465) (size 0.8) (drill 0.4) (layers "F.Cu" "B.Cu") (free) (net 13))
@@
   (via (at 65.722619 161.845) (size 0.8) (drill 0.4) (layers "F.Cu" "B.Cu") (free) (net 13))
   (via (at 200.342619 90.725) (size 0.8) (drill 0.4) (layers "F.Cu" "B.Cu") (free) (net 13))
-  (via (at 159.702619 47.545) (size 0.8) (drill 0.4) (layers "F.Cu" "B.Cu") (free) (net 13))
   (via (at 202.882619 154.225) (size 0.8) (drill 0.4) (layers "F.Cu" "B.Cu") (free) (net 13))
   (via (at 205.422619 131.365) (size 0.8) (drill 0.4) (layers "F.Cu" "B.Cu") (free) (net 13))

Commit message: Add Mounting holes for stacking PCBs
fix #8
Parts:
- added H101: StackingHole, MountingHole:MountingHole_4.3mm_M4_Pad_Via, F.Cu at (81.0, 81.0)
- added H102: StackingHole, MountingHole:MountingHole_4.3mm_M4_Pad_Via, F.Cu at (204.0, 81.0)
- added H103: StackingHole, MountingHole:MountingHole_4.3mm_M4_Pad_Via, F.Cu at (81.0, 204.0)
- added H104: StackingHole, MountingHole:MountingHole_4.3mm_M4_Pad_Via, F.Cu at (204.0, 204.0)
- renumbered H101 to H105, H102 to H106
Routing:
- net /Power/EN: track 93.4 -> 96.7 mm
- net GND: vias 5037 -> 4993

Commit message: Change DC/DC caps to MLCC
In an attempt to remove the large cap MLCC is tested.
Parts:
- added C203: 47u, Capacitor_SMD:C_1206_3216Metric_Pad1.33x1.80mm_HandSolder, F.Cu at (161.0, 82.3)
- added C204: 47u, Capacitor_SMD:C_1206_3216Metric_Pad1.33x1.80mm_HandSolder, F.Cu at (158.5, 82.3)
- C202: value 150u/50V -> 47u; footprint Capacitor_SMD:C_Elec_10x10.2 -> Capacitor_SMD:C_1206_3216Metric_Pad1.33x1.80mm_HandSolder
- moved C202 6.27 mm to (163.6, 82.3), turned to -90 degrees
- renumbered C203 to C205, C204 to C206, C205 to C207, R204 to R203, R203 to R204, TP202 to TP201, TP203 to TP202, TP201 to TP203
Routing:
- net +5V: track 1190.0 -> 1186.9 mm
- net GND: vias 4993 -> 5004

Commit message: Add solid fill to connectors
When I used a heat camera I saw that the hottest spot was
the connectors, maybe a better connection will mean a slightly
lower resistance, and therefore a lower temp
Changed lines of the file:
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@@
     (polygon
       (pts
-        (xy 245.11 245.11)
+        (xy 245.11 53.848)
+        (xy 245.11 231.14)
+        (xy 238.506 231.14)
+        (xy 238.506 244.856)
         (xy 40.005 245.11)
         (xy 40.005 40.005)
-        (xy 245.11 40.005)
+        (xy 238.506 40.005)
+        (xy 238.506 53.848)
       )
     )
@@
         (xy 174.8254 72.9536)
         (xy 181.9286 72.9536)
+      )
+    )
+  )
+  (zone (net 13) (net_name "GND") (layers F&B.Cu) (hatch edge 0.508)
+    (priority 10)
+    (connect_pads yes (clearance 0.508))
+    (min_thickness 0.254) (filled_areas_thickness no)
+    (fill yes (thermal_gap 0.508) (thermal_bridge_width 0.508))
+    (polygon
+      (pts
+        (xy 46.736 54.356)
+        (xy 40.64 54.356)
+        (xy 40.64 48.26)
+        (xy 46.736 48.26)
       )
     )
@@
         (xy 164.668 73.1996)
         (xy 166.668 73.1996)
+      )
+    )
+  )
+  (zone (net 19) (net_name "VDC") (layers F&B.Cu) (hatch edge 0.508)
+    (priority 10)
+    (connect_pads yes (clearance 0.508))
+    (min_thickness 0.254) (filled_areas_thickness no)
+    (fill yes (thermal_gap 0.508) (thermal_bridge_width 0.508))
+    (polygon
+      (pts
+        (xy 244.602 45.974)
+        (xy 237.998 45.974)
+        (xy 237.998 39.878)
+        (xy 244.602 39.878)
+      )
+    )
+  )
+  (zone (net 13) (net_name "GND") (layers F&B.Cu) (hatch edge 0.508)
+    (priority 10)
+    (connect_pads yes (clearance 0.508))
+    (min_thickness 0.254) (filled_areas_thickness no)
+    (fill yes (thermal_gap 0.508) (thermal_bridge_width 0.508))
+    (polygon
+      (pts
+        (xy 40.386 230.632)
+        (xy 46.482 230.632)
+        (xy 46.482 236.728)
+        (xy 40.386 236.728)
+      )
+    )
+  )
+  (zone (net 19) (net_name "VDC") (layers F&B.Cu) (hatch edge 0.508)
+    (priority 10)
+    (connect_pads yes (clearance 0.508))
+    (min_thickness 0.254) (filled_areas_thickness no)
+    (fill yes (thermal_gap 0.508) (thermal_bridge_width 0.508))
+    (polygon
+      (pts
+        (xy 46.736 45.974)
+        (xy 40.132 45.974)
+        (xy 40.132 39.878)
+        (xy 46.736 39.878)
       )
     )
@@
     )
   )
+  (zone (net 19) (net_name "VDC") (layers F&B.Cu) (hatch edge 0.508)
+    (priority 10)
+    (connect_pads yes (clearance 0.508))
+    (min_thickness 0.254) (filled_areas_thickness no)
+    (fill yes (thermal_gap 0.508) (thermal_bridge_width 0.508))
+    (polygon
+      (pts
+        (xy 238.252 239.014)
+        (xy 244.856 239.014)
+        (xy 244.856 245.11)
+        (xy 238.252 245.11)
+      )
+    )
+  )
   (zone (net 13) (net_name "GND") (layer "F.Cu") (hatch edge 0.508)
     (priority 7)
@@
     )
   )
+  (zone (net 13) (net_name "GND") (layer "B.Cu") (hatch edge 0.508)
+    (priority 10)
+    (connect_pads yes (clearance 0.508))
+    (min_thickness 0.254) (filled_areas_thickness no)
+    (fill yes (thermal_gap 0.508) (thermal_bridge_width 0.508))
+    (polygon
+      (pts
+        (xy 238.252 230.632)
+        (xy 244.348 230.632)
+        (xy 244.348 236.728)
+        (xy 238.252 236.728)
+      )
+    )
+  )
+  (zone (net 13) (net_name "GND") (layer "B.Cu") (hatch edge 0.508)
+    (priority 10)
+    (connect_pads yes (clearance 0.508))
+    (min_thickness 0.254) (filled_areas_thickness no)
+    (fill yes (thermal_gap 0.508) (thermal_bridge_width 0.508))
+    (polygon
+      (pts
+        (xy 244.602 54.356)
+        (xy 238.506 54.356)
+        (xy 238.506 48.26)
+        (xy 244.602 48.26)
+      )
+    )
+  )
   (zone (net 19) (net_name "VDC") (layer "B.Cu") (hatch edge 0.508)
     (priority 4)
@@
       )
     )
+  )
+  (zone (net 19) (net_name "VDC") (layer "B.Cu") (hatch edge 0.508)
+    (priority 10)
+    (connect_pads yes (clearance 0.508))
+    (min_thickness 0.254) (filled_areas_thickness no)
+    (fill yes (thermal_gap 0.508) (thermal_bridge_width 0.508))
+    (polygon
+      (pts
+        (xy 40.386 239.014)
+        (xy 46.99 239.014)
+        (xy 46.99 245.11)
+        (xy 40.386 245.11)
+      )
+    )
