File: LedWall.kicad_pcb (KiCad board)
At the start: 2 copper layers, 205 x 205 mm, 107 parts, among them J101 Conn_02x05_Odd_Even, J102 Conn_02x05_Odd_Even, J103 Conn_02x05_Odd_Even, J104 Conn_02x05_Odd_Even, U201 TPS5430DDA

Commit message: Move Testpoints that are very close to a LED
Parts:
- moved TP213 22.9 mm to (204.2, 148.8)
- moved TP218 22.9 mm to (204.2, 152.9)
- moved TP211 21.8 mm to (121.9, 67.8)
- moved TP216 21.8 mm to (121.9, 71.6)
- moved TP209 19.3 mm to (204.2, 230.6)
- moved TP214 19.3 mm to (204.2, 236.7)
- moved TP210 18.3 mm to (202.7, 177.0)
- moved TP215 18.3 mm to (202.7, 173.2)
- moved TP301 14.3 mm to (48.3, 49.3)
- moved TP307 6.18 mm to (48.3, 53.3)
- moved TP202 5.33 mm to (150.9, 82.8)
- moved TP208 5.30 mm to (146.8, 82.8)
Connections:
- TP301 pad 1: /LEDs/DataInFiltered -> /DataIn
Routing:
- net /LEDs/DataInFiltered: track 10.6 -> 4.96 mm
- net /DataIn: track 23.8 -> 21.3 mm
- net +5V: track 1186.9 -> 1189.1 mm
- net GND: vias 4972 -> 4976

Commit message: Remove components from mounting frame lines
Parts:
- moved TP207 13.4 mm to (167.6, 62.2)
- moved TP206 9.54 mm to (210.8, 48.3)
- moved C204 9.34 mm to (166.6, 77.7)
- moved C203 9.23 mm to (169.0, 77.7)
- moved C202 9.12 mm to (171.4, 77.7)
- moved C201 8.00 mm to (173.4, 71.6)
- moved C205 8.00 mm to (184.2, 75.4)
- moved D201 8.00 mm to (190.2, 74.2)
- moved U201 8.00 mm to (178.2, 76.0)
- moved C206 8.00 mm to (186.6, 75.4)
- moved L201 8.00 mm to (169.2, 71.8)
- moved TP201 8.00 mm to (167.6, 66.4)
- moved R204 7.59 mm to (176.3, 82.2)
- moved R201 7.53 mm to (174.5, 79.6)
- moved TP202 4.93 mm to (149.9, 87.6)
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Routing:
- net +5V: track 1189.1 -> 1199.0 mm
- net /Power/EN: track 96.7 -> 93.1 mm
- net GND: vias 4976 -> 4981

Commit message: Reduce board size
0.5mm have been removed from all sides
Parts:
- moved H106 6.10 mm to (233.2, 237.7)
Other:
- board size 205 x 205 mm -> 204 x 204 mm
Changed lines of the file:
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@@
   )
   (footprint "JLC:JLC_toolinghole" (layer "F.Cu")
-    (at 233.045 243.84)
+    (at 233.172 237.744)
     (property "Sheetfile" "File: LedWall.kicad_sch")
     (property "Sheetname" "")
@@
     )
   )
-  (gr_line (start 40 40) (end 40 245) (layer "Edge.Cuts") (width 0.15))
-  (gr_line (start 40 40) (end 245 40) (layer "Edge.Cuts") (width 0.15))
-  (gr_line (start 245 40) (end 245 245) (layer "Edge.Cuts") (width 0.15))
-  (gr_line (start 40 245) (end 245 245) (layer "Edge.Cuts") (width 0.15))
+  (gr_line (start 40.5 40.5) (end 40.5 244.5) (layer "Edge.Cuts") (width 0.15))
+  (gr_line (start 40.5 40.5) (end 244.5 40.5) (layer "Edge.Cuts") (width 0.15))
+  (gr_line (start 244.5 40.5) (end 244.5 244.5) (layer "Edge.Cuts") (width 0.15))
+  (gr_line (start 40.5 244.5) (end 244.5 244.5) (layer "Edge.Cuts") (width 0.15))
   (gr_text "Vin: 12V-36V" (at 227.33 41.656) (layer "B.SilkS")
     (effects (font (size 1 1) (thickness 0.15)) (justify mirror))

Commit message: Move connector up
To avoid connecting the PCBs wrong both lower pin lists
have been moved up 50 mil.
Parts:
- moved J103 1.27 mm to (45.0, 241.5)
- moved J104 1.27 mm to (242.5, 241.5)
Routing:
- net /PWR_EN: track 228.2 -> 226.4 mm
- net /DataOut: track 201.7 -> 201.1 mm
- net VDC: vias 53 -> 50
- net GND: vias 4981 -> 4910
Other:
- board text added: "LedWall rev2 2023-02-11"
- board text removed: "LedWall rev1 2022-07-21"

Commit message: Fix small changed for rev2
Other:
- board text added: "LedWall rev2 2023-03-11"
- board text removed: "LedWall rev2 2023-02-11"

Commit message: Final fixes before production
Changed lines of the file:
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@@
     (fp_line (start 1.6 0.8) (end -1.6 0.8)
       (stroke (width 0.1) (type solid)) (layer "F.Fab"))
-    (pad "1" smd roundrect (at -1.5625 0 90) (size 1.325 1.8) (layers "F.Cu" "F.Paste" "F.Mask") (roundrect_rratio 0.188679)
+    (pad "1" smd roundrect (at -1.5625 0 90) (size 1.325 1.8) (layers "F.Cu" "F.Paste" "F.Mask") (roundrect_rratio 0.1886792453)
       (net 13 "GND") (pintype "passive"))
-    (pad "2" smd roundrect (at 1.5625 0 90) (size 1.325 1.8) (layers "F.Cu" "F.Paste" "F.Mask") (roundrect_rratio 0.188679)
+    (pad "2" smd roundrect (at 1.5625 0 90) (size 1.325 1.8) (layers "F.Cu" "F.Paste" "F.Mask") (roundrect_rratio 0.1886792453)
       (net 27 "/Power/VDC+") (pintype "passive"))
     (model "${KICAD6_3DMODEL_DIR}/Capacitor_SMD.3dshapes/C_1206_3216Metric.wrl"
@@
     (fp_line (start 1.6 0.8) (end -1.6 0.8)
       (stroke (width 0.1) (type solid)) (layer "F.Fab"))
-    (pad "1" smd roundrect (at -1.5625 0 270) (size 1.325 1.8) (layers "F.Cu" "F.Paste" "F.Mask") (roundrect_rratio 0.188679)
+    (pad "1" smd roundrect (at -1.5625 0 270) (size 1.325 1.8) (layers "F.Cu" "F.Paste" "F.Mask") (roundrect_rratio 0.1886792453)
       (net 12 "+5V") (pintype "passive"))
-    (pad "2" smd roundrect (at 1.5625 0 270) (size 1.325 1.8) (layers "F.Cu" "F.Paste" "F.Mask") (roundrect_rratio 0.188679)
+    (pad "2" smd roundrect (at 1.5625 0 270) (size 1.325 1.8) (layers "F.Cu" "F.Paste" "F.Mask") (roundrect_rratio 0.1886792453)
       (net 13 "GND") (pintype "passive"))
     (model "${KICAD6_3DMODEL_DIR}/Capacitor_SMD.3dshapes/C_1206_3216Metric.wrl"
@@
     (property "Sheetfile" "LedWall.kicad_sch")
     (property "Sheetname" "")
+    (property "exclude_from_bom" "")
     (property "ki_description" "Mounting Hole without connection")
     (property "ki_keywords" "mounting hole")
-    (attr through_hole)
+    (attr through_hole exclude_from_bom)
     (fp_text reference "H106" (at -2.921 0 unlocked) (layer "F.SilkS")
         (effects (font (size 1 1) (thickness 0.15)))
@@
     (fp_line (start 1.6 0.8) (end -1.6 0.8)
       (stroke (width 0.1) (type solid)) (layer "F.Fab"))
-    (pad "1" smd roundrect (at -1.5625 0 270) (size 1.325 1.8) (layers "F.Cu" "F.Paste" "F.Mask") (roundrect_rratio 0.188679)
+    (pad "1" smd roundrect (at -1.5625 0 270) (size 1.325 1.8) (layers "F.Cu" "F.Paste" "F.Mask") (roundrect_rratio 0.1886792453)
       (net 12 "+5V") (pintype "passive"))
-    (pad "2" smd roundrect (at 1.5625 0 270) (size 1.325 1.8) (layers "F.Cu" "F.Paste" "F.Mask") (roundrect_rratio 0.188679)
+    (pad "2" smd roundrect (at 1.5625 0 270) (size 1.325 1.8) (layers "F.Cu" "F.Paste" "F.Mask") (roundrect_rratio 0.1886792453)
       (net 13 "GND") (pintype "passive"))
     (model "${KICAD6_3DMODEL_DIR}/Capacitor_SMD.3dshapes/C_1206_3216Metric.wrl"
@@
     (property "Sheetfile" "LedWall.kicad_sch")
     (property "Sheetname" "")
+    (property "exclude_from_bom" "")
     (property "ki_description" "Mounting Hole with connection")
     (property "ki_keywords" "mounting hole")
-    (attr exclude_from_pos_files)
+    (attr exclude_from_pos_files exclude_from_bom)
     (fp_text reference "H101" (at 0 -5.3) (layer "F.SilkS")
         (effects (font (size 1 1) (thickness 0.15)))
@@
     (property "Sheetfile" "LedWall.kicad_sch")
     (property "Sheetname" "")
+    (property "exclude_from_bom" "")
     (property "ki_description" "Mounting Hole with connection")
     (property "ki_keywords" "mounting hole")
-    (attr exclude_from_pos_files)
+    (attr exclude_from_pos_files exclude_from_bom)
     (fp_text reference "H102" (at 0 -5.3) (layer "F.SilkS")
         (effects (font (size 1 1) (thickness 0.15)))
@@
     (property "Sheetfile" "LedWall.kicad_sch")
     (property "Sheetname" "")
+    (property "exclude_from_bom" "")
     (property "ki_description" "Mounting Hole with connection")
     (property "ki_keywords" "mounting hole")
-    (attr exclude_from_pos_files)
+    (attr exclude_from_pos_files exclude_from_bom)
     (fp_text reference "H103" (at 0 -5.3) (layer "F.SilkS")
         (effects (font (size 1 1) (thickness 0.15)))
@@
     (fp_line (start 1.6 0.8) (end -1.6 0.8)
       (stroke (width 0.1) (type solid)) (layer "F.Fab"))
-    (pad "1" smd roundrect (at -1.5625 0 270) (size 1.325 1.8) (layers "F.Cu" "F.Paste" "F.Mask") (roundrect_rratio 0.188679)
+    (pad "1" smd roundrect (at -1.5625 0 270) (size 1.325 1.8) (layers "F.Cu" "F.Paste" "F.Mask") (roundrect_rratio 0.1886792453)
       (net 12 "+5V") (pintype "passive"))
-    (pad "2" smd roundrect (at 1.5625 0 270) (size 1.325 1.8) (layers "F.Cu" "F.Paste" "F.Mask") (roundrect_rratio 0.188679)
+    (pad "2" smd roundrect (at 1.5625 0 270) (size 1.325 1.8) (layers "F.Cu" "F.Paste" "F.Mask") (roundrect_rratio 0.1886792453)
       (net 13 "GND") (pintype "passive"))
     (model "${KICAD6_3DMODEL_DIR}/Capacitor_SMD.3dshapes/C_1206_3216Metric.wrl"
@@
     (property "Sheetfile" "LedWall.kicad_sch")
     (property "Sheetname" "")
+    (property "exclude_from_bom" "")
     (property "ki_description" "Mounting Hole with connection")
     (property "ki_keywords" "mounting hole")
-    (attr exclude_from_pos_files)
+    (attr exclude_from_pos_files exclude_from_bom)
     (fp_text reference "H104" (at 0 -5.3) (layer "F.SilkS")
         (effects (font (size 1 1) (thickness 0.15)))
@@
     (fp_line (start 1.6 0.8) (end -1.6 0.8)
       (stroke (width 0.1) (type solid)) (layer "F.Fab"))
-    (pad "1" smd roundrect (at -1.5625 0 90) (size 1.325 1.8) (layers "F.Cu" "F.Paste" "F.Mask") (roundrect_rratio 0.188679)
+    (pad "1" smd roundrect (at -1.5625 0 90) (size 1.325 1.8) (layers "F.Cu" "F.Paste" "F.Mask") (roundrect_rratio 0.1886792453)
       (net 13 "GND") (pintype "passive"))
-    (pad "2" smd roundrect (at 1.5625 0 90) (size 1.325 1.8) (layers "F.Cu" "F.Paste" "F.Mask") (roundrect_rratio 0.188679)
+    (pad "2" smd roundrect (at 1.5625 0 90) (size 1.325 1.8) (layers "F.Cu" "F.Paste" "F.Mask") (roundrect_rratio 0.1886792453)
       (net 27 "/Power/VDC+") (pintype "passive"))
     (model "${KICAD6_3DMODEL_DIR}/Capacitor_SMD.3dshapes/C_1206_3216Metric.wrl"
@@
     (property "Sheetfile" "LedWall.kicad_sch")
     (property "Sheetname" "")
+    (property "exclude_from_bom" "")
     (property "ki_description" "Mounting Hole without connection")
     (property "ki_keywords" "mounting hole")
-    (attr through_hole)
+    (attr through_hole exclude_from_bom)
     (fp_text reference "H105" (at 2.794 0 unlocked) (layer "F.SilkS")
         (effects (font (size 1 1) (thickness 0.15)))
@@
       )
     )
+  )
+  (zone (net 0) (net_name "") (layer "B.Mask") (hatch edge 0.5)
+    (connect_pads (clearance 0.508))
+    (min_thickness 0.25) (filled_areas_thickness no)
+    (fill (thermal_gap 0.5) (thermal_bridge_width 0.5))
+    (polygon
+      (pts
+        (xy 179.832 73.406)
+        (xy 176.53 73.406)
+        (xy 176.53 78.4352)
+        (xy 179.832 78.4352)
+      )
+    )
