File: LedWallPower.kicad_sch (KiCad schematic)
At the start: 15 parts, among them U1 TPS5430DDA

Commit message: Change DC/DC components and split schematic
Parts:
- added C28: 10u/50V, Capacitor_SMD:C_1206_3216Metric_Pad1.33x1.80mm_HandSolder, symbol Device:C
- C27: value 10u/50V -> 150u/50V; footprint Capacitor_SMD:C_1206_3216Metric_Pad1.33x1.80mm_HandSolder -> Capacitor_SMD:C_Elec_10x10.2; LCSC C13585 -> C72490
- L1: value 650u -> 47u; footprint Inductor_SMD:L_Bourns_SRR1208_12.7x12.7mm -> (none); LCSC C280641 -> C497841
- renumbered C28 to C29, C29 to C30
Connections:
- net GND: now also C28.1
- net VDC+: now also C28.2
Other:
- note added: "V_{in}: 10V-36V V_{out}: ~4.5V I_{out}max: 1A"
- moved on the sheet: C26, C27, C29, C30, D26, D27, L1, R3, R4, R5, R6, TP7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

Commit message: Change LED to one in JLC stock
Parts:
- L1: footprint (none) -> Ledwall:YNR6045-470M
Changed lines of the file:
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@@
     (property "Reference" "L1" (id 0) (at 193.04 47.625 90))
     (property "Value" "47u" (id 1) (at 193.04 49.9364 90))
-    (property "Footprint" "" (id 2) (at 193.04 53.34 0)
+    (property "Footprint" "Ledwall:YNR6045-470M" (id 2) (at 193.04 53.34 0)
       (effects (font (size 1.27 1.27)) hide)
     )

Commit message: Fix incorrect LCSC number for R3 and R6
Solves issue #1
Parts:
- R3, R6: LCSC C25805 -> C4184
Changed lines of the file:
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@@
       (effects (font (size 1.27 1.27)) hide)
     )
-    (property "LCSC" "C25805" (id 4) (at 215.9 57.15 0)
+    (property "LCSC" "C4184" (id 4) (at 215.9 57.15 0)
       (effects (font (size 1.27 1.27)) hide)
     )
@@
       (effects (font (size 1.27 1.27)) hide)
     )
-    (property "LCSC" "C25805" (id 4) (at 140.97 68.58 0)
+    (property "LCSC" "C4184" (id 4) (at 140.97 68.58 0)
       (effects (font (size 1.27 1.27)) hide)
     )

Commit message: Change polarity of C27
fix #5
Parts:
- C27: symbol Device:C -> Device:C_Polarized_US
Connections:
- net +5V: now also C27.1; no longer C27.2
- net GND: now also C27.2; no longer C27.1
Changed lines of the file:
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@@
     (pin "2")
   )
-  (symbol (lib_id "Device:C") (at 199.39 57.15 180) (unit 1)
+  (symbol (lib_id "Device:C_Polarized_US") (at 199.39 57.15 0) (mirror y) (unit 1)
     (in_bom yes) (on_board yes)
-    (property "Reference" "C27" (id 0) (at 202.2856 55.9816 0)
+    (property "Reference" "C27" (id 0) (at 202.2856 58.3184 0)
       (effects (font (size 1.27 1.27)) (justify right))
     )
-    (property "Value" "150u/50V" (id 1) (at 202.2856 58.293 0)
+    (property "Value" "150u/50V" (id 1) (at 202.2856 56.007 0)
       (effects (font (size 1.27 1.27)) (justify right))
     )
-    (property "Footprint" "Capacitor_SMD:C_Elec_10x10.2" (id 2) (at 198.4248 53.34 0)
+    (property "Footprint" "Capacitor_SMD:C_Elec_10x10.2" (id 2) (at 199.39 57.15 0)
       (effects (font (size 1.27 1.27)) hide)
     )

Commit message: Move 5v TP closer to DC/DC and added more TP
fix #4
Parts:
- added TP204, TP205, TP206, TP207, TP208: TestPoint, TestPoint:TestPoint_Loop_D1.80mm_Drill1.0mm_Beaded, symbol Connector:TestPoint
- renumbered C26 to C201, C27 to C202, C28 to C203, C29 to C204, C30 to C205, D26 to D201, D27 to D202, L1 to L201, R3 to R201, R4 to R202, R5 to R203, R6 to R204, TP7 to TP201, TP8 to TP202, TP9 to TP203, U1 to U201
Connections:
- net +5V: now also TP204.1, TP205.1, TP206.1, TP207.1, TP208.1

Commit message: Add GND testpoints
Each other testpoint now has its own ground reference

fix #6
Parts:
- added TP204, TP205, TP206, TP212, TP213, TP214, TP215, TP216: TestPoint, TestPoint:TestPoint_Loop_D1.80mm_Drill1.0mm_Beaded, symbol Connector:TestPoint
- renumbered TP204 to TP207, TP205 to TP208, TP206 to TP209, TP207 to TP210, TP208 to TP211
Connections:
- net GND: now also TP204.1, TP205.1, TP206.1, TP212.1, TP213.1, TP214.1, TP215.1, TP216.1

Commit message: Add 12V testpoint
fix #3
Parts:
- added TP201, TP205: TestPoint, TestPoint:TestPoint_Loop_D1.80mm_Drill1.0mm_Beaded, symbol Connector:TestPoint
- renumbered TP201 to TP202, TP202 to TP203, TP203 to TP204, TP204 to TP207, TP205 to TP208, TP207 to TP209, TP208 to TP210, TP209 to TP211, TP210 to TP212, TP211 to TP213, TP212 to TP214, TP213 to TP215, TP214 to TP216, TP215 to TP217, TP216 to TP218
Connections:
- net GND: now also TP205.1
- net VDC: now also TP201.1
Changed lines of the file:
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@@
   (junction (at 99.06 53.34) (diameter 0) (color 0 0 0 0)
   )
+  (junction (at 99.06 73.66) (diameter 0) (color 0 0 0 0)
+  )
   (junction (at 215.9 53.34) (diameter 0) (color 0 0 0 0)
   )
@@
   (junction (at 124.46 177.8) (diameter 0) (color 0 0 0 0)
   )
+  (junction (at 81.28 53.34) (diameter 0) (color 0 0 0 0)
+  )
   (junction (at 124.46 190.5) (diameter 0) (color 0 0 0 0)
   )
@@
     (stroke (width 0) (type default) (color 0 0 0 0))
   )
-  (wire (pts (xy 83.185 53.34) (xy 83.185 48.26))
+  (wire (pts (xy 76.2 53.34) (xy 76.2 48.26))
     (stroke (width 0) (type default) (color 0 0 0 0))
   )
@@
     (stroke (width 0) (type default) (color 0 0 0 0))
   )
+  (wire (pts (xy 81.28 53.34) (xy 76.2 53.34))
+    (stroke (width 0) (type default) (color 0 0 0 0))
+  )
   (wire (pts (xy 111.76 177.8) (xy 99.06 177.8))
     (stroke (width 0) (type default) (color 0 0 0 0))
@@
     (stroke (width 0) (type default) (color 0 0 0 0))
   )
+  (wire (pts (xy 81.28 73.66) (xy 99.06 73.66))
+    (stroke (width 0) (type default) (color 0 0 0 0))
+  )
   (wire (pts (xy 111.76 190.5) (xy 99.06 190.5))
     (stroke (width 0) (type default) (color 0 0 0 0))
@@
     (stroke (width 0) (type default) (color 0 0 0 0))
   )
-  (wire (pts (xy 85.09 53.34) (xy 83.185 53.34))
+  (wire (pts (xy 81.28 53.34) (xy 85.09 53.34))
     (stroke (width 0) (type default) (color 0 0 0 0))
   )
@@
     (pin "9")
   )
-  (symbol (lib_id "power:VDC") (at 83.185 48.26 0) (unit 1)
-    (in_bom yes) (on_board yes)
-    (property "Reference" "#PWR0201" (id 0) (at 83.185 50.8 0)
-      (effects (font (size 1.27 1.27)) hide)
-    )
-    (property "Value" "VDC" (id 1) (at 83.566 43.8658 0))
-    (property "Footprint" "" (id 2) (at 83.185 48.26 0)
-      (effects (font (size 1.27 1.27)) hide)
-    )
-    (property "Datasheet" "" (id 3) (at 83.185 48.26 0)
+  (symbol (lib_id "power:VDC") (at 76.2 48.26 0) (unit 1)
+    (in_bom yes) (on_board yes)
+    (property "Reference" "#PWR0201" (id 0) (at 76.2 50.8 0)
+      (effects (font (size 1.27 1.27)) hide)
+    )
+    (property "Value" "VDC" (id 1) (at 76.581 43.8658 0))
+    (property "Footprint" "" (id 2) (at 76.2 48.26 0)
+      (effects (font (size 1.27 1.27)) hide)
+    )
+    (property "Datasheet" "" (id 3) (at 76.2 48.26 0)
       (effects (font (size 1.27 1.27)) hide)
     )
@@
   (symbol (lib_id "power:GND") (at 152.4 74.93 0) (unit 1)
     (in_bom yes) (on_board yes)
-    (property "Reference" "#PWR0205" (id 0) (at 152.4 81.28 0)
+    (property "Reference" "#PWR0204" (id 0) (at 152.4 81.28 0)
       (effects (font (size 1.27 1.27)) hide)
     )
@@
   (symbol (lib_id "power:GND") (at 215.9 80.01 0) (unit 1)
     (in_bom yes) (on_board yes)
-    (property "Reference" "#PWR0204" (id 0) (at 215.9 86.36 0)
+    (property "Reference" "#PWR0205" (id 0) (at 215.9 86.36 0)
       (effects (font (size 1.27 1.27)) hide)
     )
@@
   (symbol (lib_id "Connector:TestPoint") (at 135.89 63.5 0) (unit 1)
     (in_bom yes) (on_board yes) (fields_autoplaced)
-    (property "Reference" "TP203" (id 0) (at 137.287 59.3633 0)
+    (property "Reference" "TP204" (id 0) (at 137.287 59.3633 0)
       (effects (font (size 1.27 1.27)) (justify left))
     )
@@
   (symbol (lib_id "Connector:TestPoint") (at 124.46 175.26 0) (unit 1)
     (in_bom yes) (on_board yes) (fields_autoplaced)
-    (property "Reference" "TP209" (id 0) (at 125.857 171.1233 0)
+    (property "Reference" "TP211" (id 0) (at 125.857 171.1233 0)
       (effects (font (size 1.27 1.27)) (justify left))
     )
@@
   (symbol (lib_id "Connector:TestPoint") (at 111.76 175.26 0) (unit 1)
     (in_bom yes) (on_board yes) (fields_autoplaced)
-    (property "Reference" "TP208" (id 0) (at 113.157 171.1233 0)
+    (property "Reference" "TP210" (id 0) (at 113.157 171.1233 0)
       (effects (font (size 1.27 1.27)) (justify left))
     )
@@
   (symbol (lib_id "Connector:TestPoint") (at 182.88 53.34 0) (unit 1)
     (in_bom yes) (on_board yes) (fields_autoplaced)
-    (property "Reference" "TP201" (id 0) (at 184.277 49.2033 0)
+    (property "Reference" "TP202" (id 0) (at 184.277 49.2033 0)
       (effects (font (size 1.27 1.27)) (justify left))
     )
@@
   (symbol (lib_id "Connector:TestPoint") (at 137.16 175.26 0) (unit 1)
     (in_bom yes) (on_board yes) (fields_autoplaced)
-    (property "Reference" "TP210" (id 0) (at 138.557 171.1233 0)
+    (property "Reference" "TP212" (id 0) (at 138.557 171.1233 0)
       (effects (font (size 1.27 1.27)) (justify left))
     )
@@
   (symbol (lib_id "Connector:TestPoint") (at 99.06 175.26 0) (unit 1)
     (in_bom yes) (on_board yes) (fields_autoplaced)
-    (property "Reference" "TP207" (id 0) (at 100.457 171.1233 0)
+    (property "Reference" "TP209" (id 0) (at 100.457 171.1233 0)
       (effects (font (size 1.27 1.27)) (justify left))
     )
@@
     (pin "2")
   )
+  (symbol (lib_id "Connector:TestPoint") (at 81.28 53.34 0) (unit 1)
+    (in_bom yes) (on_board yes) (fields_autoplaced)
+    (property "Reference" "TP201" (id 0) (at 82.677 50.4718 0)
+      (effects (font (size 1.27 1.27)) (justify left))
+    )
+    (property "Value" "TestPoint" (id 1) (at 82.677 51.7402 0)
+      (effects (font (size 1.27 1.27)) (justify left) hide)
+    )
+    (property "Footprint" "TestPoint:TestPoint_Loop_D1.80mm_Drill1.0mm_Beaded" (id 2) (at 86.36 53.34 0)
+      (effects (font (size 1.27 1.27)) hide)
+    )
+    (property "Datasheet" "~" (id 3) (at 86.36 53.34 0)
+      (effects (font (size 1.27 1.27)) hide)
+    )
+    (property "LCSC" "C238122" (id 4) (at 81.28 53.34 0)
+      (effects (font (size 1.27 1.27)) hide)
+    )
+    (pin "1")
+  )
   (symbol (lib_id "Device:R") (at 130.81 63.5 90) (unit 1)
     (in_bom yes) (on_board yes)
@@
   (symbol (lib_id "Connector:TestPoint") (at 99.06 187.96 0) (unit 1)
     (in_bom yes) (on_board yes) (fields_autoplaced)
-    (property "Reference" "TP212" (id 0) (at 100.457 183.8233 0)
+    (property "Reference" "TP214" (id 0) (at 100.457 183.8233 0)
       (effects (font (size 1.27 1.27)) (justify left))
     )
@@
   (symbol (lib_id "Connector:TestPoint") (at 199.39 53.34 0) (unit 1)
     (in_bom yes) (on_board yes) (fields_autoplaced)
-    (property "Reference" "TP202" (id 0) (at 200.787 49.2033 0)
+    (property "Reference" "TP203" (id 0) (at 200.787 49.2033 0)
       (effects (font (size 1.27 1.27)) (justify left))
     )
@@
   (symbol (lib_id "Connector:TestPoint") (at 137.16 187.96 0) (unit 1)
     (in_bom yes) (on_board yes) (fields_autoplaced)
-    (property "Reference" "TP215" (id 0) (at 138.557 183.8233 0)
+    (property "Reference" "TP217" (id 0) (at 138.557 183.8233 0)
       (effects (font (size 1.27 1.27)) (justify left))
     )
@@
   (symbol (lib_id "Connector:TestPoint") (at 124.46 187.96 0) (unit 1)
     (in_bom yes) (on_board yes) (fields_autoplaced)
-    (property "Reference" "TP214" (id 0) (at 125.857 183.8233 0)
+    (property "Reference" "TP216" (id 0) (at 125.857 183.8233 0)
       (effects (font (size 1.27 1.27)) (justify left))
     )
@@
     (pin "1")
   )
+  (symbol (lib_id "Connector:TestPoint") (at 81.28 73.66 180) (unit 1)
+    (in_bom yes) (on_board yes) (fields_autoplaced)
+    (property "Reference" "TP205" (id 0) (at 82.677 77.3958 0)
+      (effects (font (size 1.27 1.27)) (justify right))
+    )
+    (property "Value" "TestPoint" (id 1) (at 79.883 75.2598 0)
+      (effects (font (size 1.27 1.27)) (justify left) hide)
+    )
+    (property "Footprint" "TestPoint:TestPoint_Loop_D1.80mm_Drill1.0mm_Beaded" (id 2) (at 76.2 73.66 0)
+      (effects (font (size 1.27 1.27)) hide)
+    )
+    (property "Datasheet" "~" (id 3) (at 76.2 73.66 0)
+      (effects (font (size 1.27 1.27)) hide)
+    )
+    (property "LCSC" "C238122" (id 4) (at 81.28 73.66 0)
+      (effects (font (size 1.27 1.27)) hide)
+    )
+    (pin "1")
+  )
   (symbol (lib_id "power:GND") (at 162.56 193.04 0) (unit 1)
     (in_bom yes) (on_board yes)
@@
   (symbol (lib_id "Connector:TestPoint") (at 149.86 175.26 0) (unit 1)
     (in_bom yes) (on_board yes) (fields_autoplaced)
-    (property "Reference" "TP211" (id 0) (at 151.257 171.1233 0)
+    (property "Reference" "TP213" (id 0) (at 151.257 171.1233 0)
       (effects (font (size 1.27 1.27)) (justify left))
     )
@@
   (symbol (lib_id "Connector:TestPoint") (at 199.39 77.47 0) (unit 1)
     (in_bom yes) (on_board yes) (fields_autoplaced)
-    (property "Reference" "TP205" (id 0) (at 200.787 74.6018 0)
+    (property "Reference" "TP208" (id 0) (at 200.787 74.6018 0)
       (effects (font (size 1.27 1.27)) (justify left))
     )
@@
   (symbol (lib_id "Connector:TestPoint") (at 149.86 187.96 0) (unit 1)
     (in_bom yes) (on_board yes) (fields_autoplaced)
-    (property "Reference" "TP216" (id 0) (at 151.257 183.8233 0)
+    (property "Reference" "TP218" (id 0) (at 151.257 183.8233 0)
       (effects (font (size 1.27 1.27)) (justify left))
     )
@@
   (symbol (lib_id "Connector:TestPoint") (at 182.88 77.47 0) (unit 1)
     (in_bom yes) (on_board yes) (fields_autoplaced)
-    (property "Reference" "TP204" (id 0) (at 184.277 74.6018 0)
+    (property "Reference" "TP207" (id 0) (at 184.277 74.6018 0)
       (effects (font (size 1.27 1.27)) (justify left))
     )
@@
   (symbol (lib_id "Connector:TestPoint") (at 111.76 187.96 0) (unit 1)
     (in_bom yes) (on_board yes) (fields_autoplaced)
-    (property "Reference" "TP213" (id 0) (at 113.157 183.8233 0)
-      (effects (font (size 1.27 1.27)) (justify left))
-    )
+    (property "Reference" "TP215" (id 0) (at 113.157 183.8233 0)
+      (effects (font (size 1.27 1.27)) (justify left))
+    )

Commit message: Add some more requirements
Other:
- note added: "Reqs: Vin 12-36V Enable pulled down Enable series resistor to limit current draw on enable pin Output close to 5V > 1.5A output"
Changed lines of the file:
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@@
+    (stroke (width 0) (type default) (color 0 0 0 0))
+  )
+  (polyline (pts (xy 177.8 152.4) (xy 284.48 152.4))
     (stroke (width 0) (type default) (color 0 0 0 0))
   )
@@
     (effects (font (size 1.27 1.27)) (justify left bottom))
   )
+  (text "Reqs:\nVin 12-36V\nEnable pulled down\nEnable series resistor to limit current draw on enable pin\nOutput close to 5V\n> 1.5A output"
+    (at 180.34 165.1 0)
+    (effects (font (size 1.27 1.27)) (justify left bottom))
+  )
