File: LedWall.kicad_sch (KiCad schematic)
At the start: 64 parts, among them J1 Conn_02x05_Odd_Even, J2 Conn_02x05_Odd_Even, J3 Conn_02x05_Odd_Even, J4 Conn_02x05_Odd_Even

Commit message: Change DC/DC components and split schematic
Parts:
- removed C1, C10, C11, C12, C13, C14, C15, C16, C17, C18, C19, C2, C20, C21, C22, C23, C24, C25, C3, C4, C5, C6, C7, C8, C9: 100n/10V, Capacitor_SMD:C_0603_1608Metric_Pad1.08x0.95mm_HandSolder, symbol Device:C
- removed D1, D10, D11, D12, D13, D14, D15, D16, D17, D18, D19, D2, D20, D21, D22, D23, D24, D25, D3, D4, D5, D6, D7, D8, D9: WS2812B, LED_SMD:LED_WS2812B_PLCC4_5.0x5.0mm_P3.2mm, symbol LED:WS2812B
- removed R1: 22, Resistor_SMD:R_0603_1608Metric_Pad0.98x0.95mm_HandSolder, symbol Device:R
- removed R2: 20k, Resistor_SMD:R_0603_1608Metric_Pad0.98x0.95mm_HandSolder, symbol Device:R
- removed TP1, TP2, TP3, TP4, TP5, TP6: TestPoint, TestPoint:TestPoint_Loop_D1.80mm_Drill1.0mm_Beaded, symbol Connector:TestPoint
Other:
- sheet Led Wall Power renamed Power
- added sheet LEDs (leds.kicad_sch)
- moved on the sheet: H1, H2

Commit message: Move 5v TP closer to DC/DC and added more TP
fix #4
Parts:
- renumbered H1 to H101, H2 to H102, J1 to J101, J2 to J102, J3 to J103, J4 to J104

Commit message: Add some more requirements
Other:
- note added: "Reqs: 4 pins for every power connection 2 pins for every signal connection"
- note removed: "Reqs: Vin 12-36V"
- moved on the sheet: H101, H102
Changed lines of the file:
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@@
+    (stroke (width 0) (type default) (color 0 0 0 0))
+  )
+  (polyline (pts (xy 176.53 166.37) (xy 101.6 166.37))
     (stroke (width 0) (type default) (color 0 0 0 0))
   )
@@
     (stroke (width 0) (type default) (color 0 0 0 0))
   )
+  (polyline (pts (xy 101.6 166.37) (xy 101.6 196.85))
+    (stroke (width 0) (type default) (color 0 0 0 0))
+  )
   (wire (pts (xy 267.97 105.41) (xy 267.97 107.95))
     (stroke (width 0) (type default) (color 0 0 0 0))
@@
     (stroke (width 0) (type default) (color 0 0 0 0))
   )
-  (text "Reqs:\nVin 12-36V" (at 19.05 182.88 0)
+  (text "Reqs:\n4 pins for every power connection\n2 pins for every signal connection"
+    (at 19.05 182.88 0)
     (effects (font (size 1.27 1.27)) (justify left bottom))
   )
@@
     (pin "1")
   )
-  (symbol (lib_id "Mechanical:MountingHole") (at 137.16 121.92 0) (unit 1)
+  (symbol (lib_id "Mechanical:MountingHole") (at 132.08 177.8 0) (unit 1)
     (in_bom yes) (on_board yes) (fields_autoplaced)
-    (property "Reference" "H102" (id 0) (at 139.7 121.0853 0)
+    (property "Reference" "H102" (id 0) (at 134.62 176.9653 0)
       (effects (font (size 1.27 1.27)) (justify left))
     )
-    (property "Value" "ToolingHole" (id 1) (at 139.7 123.6222 0)
+    (property "Value" "ToolingHole" (id 1) (at 134.62 179.5022 0)
       (effects (font (size 1.27 1.27)) (justify left))
     )
-    (property "Footprint" "JLC:JLC_toolinghole" (id 2) (at 137.16 121.92 0)
-      (effects (font (size 1.27 1.27)) hide)
-    )
-    (property "Datasheet" "~" (id 3) (at 137.16 121.92 0)
-      (effects (font (size 1.27 1.27)) hide)
-    )
-  )
-  (symbol (lib_id "Mechanical:MountingHole") (at 116.84 121.92 270) (unit 1)
-    (in_bom yes) (on_board yes)
-    (property "Reference" "H101" (id 0) (at 119.38 121.0853 90)
+    (property "Footprint" "JLC:JLC_toolinghole" (id 2) (at 132.08 177.8 0)
+      (effects (font (size 1.27 1.27)) hide)
+    )
+    (property "Datasheet" "~" (id 3) (at 132.08 177.8 0)
+      (effects (font (size 1.27 1.27)) hide)
+    )
+  )
+  (symbol (lib_id "Mechanical:MountingHole") (at 111.76 177.8 270) (unit 1)
+    (in_bom yes) (on_board yes)
+    (property "Reference" "H101" (id 0) (at 114.3 176.9653 90)
       (effects (font (size 1.27 1.27)) (justify left))
     )
-    (property "Value" "ToolingHole" (id 1) (at 119.38 123.6222 90)
+    (property "Value" "ToolingHole" (id 1) (at 114.3 179.5022 90)
       (effects (font (size 1.27 1.27)) (justify left))
     )
-    (property "Footprint" "JLC:JLC_toolinghole" (id 2) (at 116.84 121.92 0)
-      (effects (font (size 1.27 1.27)) hide)
-    )
-    (property "Datasheet" "~" (id 3) (at 116.84 121.92 0)
-      (effects (font (size 1.27 1.27)) hide)
-    )
+    (property "Footprint" "JLC:JLC_toolinghole" (id 2) (at 111.76 177.8 0)
+      (effects (font (size 1.27 1.27)) hide)
+    )
+    (property "Datasheet" "~" (id 3) (at 111.76 177.8 0)
+      (effects (font (size 1.27 1.27)) hide)
+    )

Commit message: Add Mounting holes for stacking PCBs
fix #8
Parts:
- added H101, H102, H103, H104: StackingHole, symbol Mechanical:MountingHole_Pad
- renumbered H101 to H105, H102 to H106
Connections:
- net GND: now also H101.1, H102.1, H103.1, H104.1
Other:
- note added: "Reqs: 4 pins for every power connection 2 pins for every signal connection 2 tooling holes needed for Assembly 4 stacking holes needed to be able to stack boards"
- note removed: "Reqs: 4 pins for every power connection 2 pins for every signal connection"
Changed lines of the file:
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@@
   (junction (at 242.57 49.53) (diameter 0) (color 0 0 0 0)
   )
+  (junction (at 195.58 149.86) (diameter 0) (color 0 0 0 0)
+  )
+  (junction (at 236.22 149.86) (diameter 0) (color 0 0 0 0)
+  )
   (junction (at 267.97 59.69) (diameter 0) (color 0 0 0 0)
   )
@@
   (junction (at 267.97 25.4) (diameter 0) (color 0 0 0 0)
   )
+  (junction (at 215.9 149.86) (diameter 0) (color 0 0 0 0)
+  )
   (junction (at 267.97 107.95) (diameter 0) (color 0 0 0 0)
   )
@@
     (stroke (width 0) (type default) (color 0 0 0 0))
   )
+  (wire (pts (xy 195.58 144.78) (xy 195.58 149.86))
+    (stroke (width 0) (type default) (color 0 0 0 0))
+  )
   (wire (pts (xy 261.62 33.02) (xy 267.97 33.02))
     (stroke (width 0) (type default) (color 0 0 0 0))
@@
     (stroke (width 0) (type default) (color 0 0 0 0))
   )
+  (wire (pts (xy 215.9 144.78) (xy 215.9 149.86))
+    (stroke (width 0) (type default) (color 0 0 0 0))
+  )
   (wire (pts (xy 242.57 25.4) (xy 233.68 25.4))
     (stroke (width 0) (type default) (color 0 0 0 0))
@@
     (stroke (width 0) (type default) (color 0 0 0 0))
   )
+  (wire (pts (xy 215.9 149.86) (xy 195.58 149.86))
+    (stroke (width 0) (type default) (color 0 0 0 0))
+  )
   (wire (pts (xy 248.92 54.61) (xy 240.03 54.61))
     (stroke (width 0) (type default) (color 0 0 0 0))
@@
     (stroke (width 0) (type default) (color 0 0 0 0))
   )
+  (wire (pts (xy 195.58 149.86) (xy 195.58 154.94))
+    (stroke (width 0) (type default) (color 0 0 0 0))
+  )
   (wire (pts (xy 35.56 49.53) (xy 43.18 49.53))
     (stroke (width 0) (type default) (color 0 0 0 0))
@@
     (stroke (width 0) (type default) (color 0 0 0 0))
   )
+  (wire (pts (xy 256.54 144.78) (xy 256.54 149.86))
+    (stroke (width 0) (type default) (color 0 0 0 0))
+  )
   (wire (pts (xy 248.92 105.41) (xy 242.57 105.41))
     (stroke (width 0) (type default) (color 0 0 0 0))
@@
     (stroke (width 0) (type default) (color 0 0 0 0))
   )
+  (wire (pts (xy 236.22 149.86) (xy 215.9 149.86))
+    (stroke (width 0) (type default) (color 0 0 0 0))
+  )
   (wire (pts (xy 35.56 35.56) (xy 43.18 35.56))
     (stroke (width 0) (type default) (color 0 0 0 0))
   )
+  (wire (pts (xy 256.54 149.86) (xy 236.22 149.86))
+    (stroke (width 0) (type default) (color 0 0 0 0))
+  )
   (wire (pts (xy 248.92 102.87) (xy 241.3 102.87))
     (stroke (width 0) (type default) (color 0 0 0 0))
@@
     (stroke (width 0) (type default) (color 0 0 0 0))
   )
+  (wire (pts (xy 236.22 144.78) (xy 236.22 149.86))
+    (stroke (width 0) (type default) (color 0 0 0 0))
+  )
   (wire (pts (xy 248.92 57.15) (xy 242.57 57.15))
     (stroke (width 0) (type default) (color 0 0 0 0))
@@
     (stroke (width 0) (type default) (color 0 0 0 0))
   )
+  (polyline (pts (xy 284.48 132.08) (xy 177.8 132.08))
+    (stroke (width 0) (type default) (color 0 0 0 0))
+  )
   (wire (pts (xy 62.23 35.56) (xy 64.77 35.56))
     (stroke (width 0) (type default) (color 0 0 0 0))
@@
     (stroke (width 0) (type default) (color 0 0 0 0))
   )
-  (text "Reqs:\n4 pins for every power connection\n2 pins for every signal connection"
+  (polyline (pts (xy 177.8 132.08) (xy 177.8 165.1))
+    (stroke (width 0) (type default) (color 0 0 0 0))
+  )
+  (text "Reqs:\n4 pins for every power connection\n2 pins for every signal connection\n2 tooling holes needed for Assembly\n4 stacking holes needed to be able to stack boards"
     (at 19.05 182.88 0)
     (effects (font (size 1.27 1.27)) (justify left bottom))
@@
     (pin "1")
   )
+  (symbol (lib_id "power:GND") (at 195.58 154.94 0) (unit 1)
+    (in_bom yes) (on_board yes)
+    (property "Reference" "#PWR?" (id 0) (at 195.58 161.29 0)
+      (effects (font (size 1.27 1.27)) hide)
+    )
+    (property "Value" "GND" (id 1) (at 195.707 159.3342 0))
+    (property "Footprint" "" (id 2) (at 195.58 154.94 0)
+      (effects (font (size 1.27 1.27)) hide)
+    )
+    (property "Datasheet" "" (id 3) (at 195.58 154.94 0)
+      (effects (font (size 1.27 1.27)) hide)
+    )
+    (pin "1")
+  )
+  (symbol (lib_id "Mechanical:MountingHole_Pad") (at 256.54 142.24 0) (unit 1)
+    (in_bom yes) (on_board yes) (fields_autoplaced)
+    (property "Reference" "H104" (id 0) (at 259.08 140.1353 0)
+      (effects (font (size 1.27 1.27)) (justify left))
+    )
+    (property "Value" "StackingHole" (id 1) (at 259.08 142.6722 0)
+      (effects (font (size 1.27 1.27)) (justify left))
+    )
+    (property "Footprint" "" (id 2) (at 256.54 142.24 0)
+      (effects (font (size 1.27 1.27)) hide)
+    )
+    (property "Datasheet" "~" (id 3) (at 256.54 142.24 0)
+      (effects (font (size 1.27 1.27)) hide)
+    )
+    (pin "1")
+  )
   (symbol (lib_id "Mechanical:MountingHole") (at 132.08 177.8 0) (unit 1)
     (in_bom yes) (on_board yes) (fields_autoplaced)
-    (property "Reference" "H102" (id 0) (at 134.62 176.9653 0)
+    (property "Reference" "H106" (id 0) (at 134.62 176.9653 0)
       (effects (font (size 1.27 1.27)) (justify left))
     )
@@
     )
   )
+  (symbol (lib_id "Mechanical:MountingHole_Pad") (at 236.22 142.24 0) (unit 1)
+    (in_bom yes) (on_board yes) (fields_autoplaced)
+    (property "Reference" "H103" (id 0) (at 238.76 140.1353 0)
+      (effects (font (size 1.27 1.27)) (justify left))
+    )
+    (property "Value" "StackingHole" (id 1) (at 238.76 142.6722 0)
+      (effects (font (size 1.27 1.27)) (justify left))
+    )
+    (property "Footprint" "" (id 2) (at 236.22 142.24 0)
+      (effects (font (size 1.27 1.27)) hide)
+    )
+    (property "Datasheet" "~" (id 3) (at 236.22 142.24 0)
+      (effects (font (size 1.27 1.27)) hide)
+    )
+    (pin "1")
+  )
+  (symbol (lib_id "Mechanical:MountingHole_Pad") (at 215.9 142.24 0) (unit 1)
+    (in_bom yes) (on_board yes)
+    (property "Reference" "H102" (id 0) (at 218.44 140.1353 0)
+      (effects (font (size 1.27 1.27)) (justify left))
+    )
+    (property "Value" "StackingHole" (id 1) (at 218.44 142.6722 0)
+      (effects (font (size 1.27 1.27)) (justify left))
+    )
+    (property "Footprint" "" (id 2) (at 215.9 142.24 0)
+      (effects (font (size 1.27 1.27)) hide)
+    )
+    (property "Datasheet" "~" (id 3) (at 215.9 142.24 0)
+      (effects (font (size 1.27 1.27)) hide)
+    )
+    (pin "1")
+  )
+  (symbol (lib_id "Mechanical:MountingHole_Pad") (at 195.58 142.24 0) (unit 1)
+    (in_bom yes) (on_board yes) (fields_autoplaced)
+    (property "Reference" "H101" (id 0) (at 198.12 140.1353 0)
+      (effects (font (size 1.27 1.27)) (justify left))
+    )
+    (property "Value" "StackingHole" (id 1) (at 198.12 142.6722 0)
+      (effects (font (size 1.27 1.27)) (justify left))
+    )
+    (property "Footprint" "" (id 2) (at 195.58 142.24 0)
+      (effects (font (size 1.27 1.27)) hide)
+    )
+    (property "Datasheet" "~" (id 3) (at 195.58 142.24 0)
+      (effects (font (size 1.27 1.27)) hide)
+    )
+    (pin "1")
+  )
   (symbol (lib_id "Mechanical:MountingHole") (at 111.76 177.8 270) (unit 1)
     (in_bom yes) (on_board yes)
-    (property "Reference" "H101" (id 0) (at 114.3 176.9653 90)
+    (property "Reference" "H105" (id 0) (at 114.3 176.9653 90)
       (effects (font (size 1.27 1.27)) (justify left))
     )
@@
       (reference "#PWR0402") (unit 1) (value "GND") (footprint "")
     )
+    (path "/15e69da9-56c0-4854-8649-7e068449124a"
+      (reference "#PWR?") (unit 1) (value "GND") (footprint "")
+    )
     (path "/00000000-0000-0000-0000-000060250caf/00000000-0000-0000-0000-00006026c80b"
       (reference "C201") (unit 1) (value "10n") (footprint "Capacitor_SMD:C_0603_1608Metric_Pad1.08x0.95mm_HandSolder")
@@
       (reference "D325") (unit 1) (value "WS2812B") (footprint "LED_SMD:LED_WS2812B_PLCC4_5.0x5.0mm_P3.2mm")
     )
+    (path "/c683f6ce-10d2-4700-ac6d-4c1aaad73b42"
+      (reference "H101") (unit 1) (value "StackingHole") (footprint "")
+    )
+    (path "/5d07e589-af55-4d48-811f-40d4db0274a2"
+      (reference "H102") (unit 1) (value "StackingHole") (footprint "")
+    )
+    (path "/527554b9-fdf1-4700-a5a2-8ea608d514cc"
+      (reference "H103") (unit 1) (value "StackingHole") (footprint "")
+    )
+    (path "/211b24fb-4a86-4015-98e8-23eec98f28b8"
+      (reference "H104") (unit 1) (value "StackingHole") (footprint "")
+    )
     (path "/ebda81a3-b2be-4646-827f-a3500dfd9585"
-      (reference "H101") (unit 1) (value "ToolingHole") (footprint "JLC:JLC_toolinghole")
+      (reference "H105") (unit 1) (value "ToolingHole") (footprint "JLC:JLC_toolinghole")
     )
     (path "/3980be34-4222-43f0-ab80-83a36807e8c3"
-      (reference "H102") (unit 1) (value "ToolingHole") (footprint "JLC:JLC_toolinghole")
+      (reference "H106") (unit 1) (value "ToolingHole") (footprint "JLC:JLC_toolinghole")
     )
     (path "/00000000-0000-0000-0000-00006016f1d9"
