File: LedWall.kicad_sch (KiCad schematic)
At the start: 10 parts, among them J101 Conn_02x05_Odd_Even, J102 Conn_02x05_Odd_Even, J103 Conn_02x05_Odd_Even, J104 Conn_02x05_Odd_Even

Commit message: Move Testpoints that are very close to a LED
Parts:
- H101, H102, H103, H104: footprint (none) -> MountingHole:MountingHole_4.3mm_M4_Pad_Via
Changed lines of the file:
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@@
       (effects (font (size 1.27 1.27)) (justify left))
     )
-    (property "Footprint" "" (id 2) (at 256.54 142.24 0)
+    (property "Footprint" "MountingHole:MountingHole_4.3mm_M4_Pad_Via" (id 2) (at 256.54 142.24 0)
       (effects (font (size 1.27 1.27)) hide)
     )
@@
       (effects (font (size 1.27 1.27)) (justify left))
     )
-    (property "Footprint" "" (id 2) (at 236.22 142.24 0)
+    (property "Footprint" "MountingHole:MountingHole_4.3mm_M4_Pad_Via" (id 2) (at 236.22 142.24 0)
       (effects (font (size 1.27 1.27)) hide)
     )
@@
       (effects (font (size 1.27 1.27)) (justify left))
     )
-    (property "Footprint" "" (id 2) (at 215.9 142.24 0)
+    (property "Footprint" "MountingHole:MountingHole_4.3mm_M4_Pad_Via" (id 2) (at 215.9 142.24 0)
       (effects (font (size 1.27 1.27)) hide)
     )
@@
       (effects (font (size 1.27 1.27)) (justify left))
     )
-    (property "Footprint" "" (id 2) (at 195.58 142.24 0)
+    (property "Footprint" "MountingHole:MountingHole_4.3mm_M4_Pad_Via" (id 2) (at 195.58 142.24 0)
       (effects (font (size 1.27 1.27)) hide)
     )
@@
     )
     (path "/c683f6ce-10d2-4700-ac6d-4c1aaad73b42"
-      (reference "H101") (unit 1) (value "StackingHole") (footprint "")
+      (reference "H101") (unit 1) (value "StackingHole") (footprint "MountingHole:MountingHole_4.3mm_M4_Pad_Via")
     )
     (path "/5d07e589-af55-4d48-811f-40d4db0274a2"
-      (reference "H102") (unit 1) (value "StackingHole") (footprint "")
+      (reference "H102") (unit 1) (value "StackingHole") (footprint "MountingHole:MountingHole_4.3mm_M4_Pad_Via")
     )
     (path "/527554b9-fdf1-4700-a5a2-8ea608d514cc"
-      (reference "H103") (unit 1) (value "StackingHole") (footprint "")
+      (reference "H103") (unit 1) (value "StackingHole") (footprint "MountingHole:MountingHole_4.3mm_M4_Pad_Via")
     )
     (path "/211b24fb-4a86-4015-98e8-23eec98f28b8"
-      (reference "H104") (unit 1) (value "StackingHole") (footprint "")
+      (reference "H104") (unit 1) (value "StackingHole") (footprint "MountingHole:MountingHole_4.3mm_M4_Pad_Via")
     )
     (path "/ebda81a3-b2be-4646-827f-a3500dfd9585"

Commit message: Final fixes before production
Parts:
- H101, H102, H103, H104, H105, H106: now left out of the parts list
Other:
- moved on the sheet: H105, H106
Changed lines of the file:
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@@
   )
   (symbol (lib_id "Mechanical:MountingHole_Pad") (at 256.54 142.24 0) (unit 1)
-    (in_bom yes) (on_board yes) (dnp no) (fields_autoplaced)
+    (in_bom no) (on_board yes) (dnp no) (fields_autoplaced)
     (property "Reference" "H104" (at 259.08 140.1353 0)
       (effects (font (size 1.27 1.27)) (justify left))
@@
     )
   )
-  (symbol (lib_id "Mechanical:MountingHole") (at 132.08 177.8 0) (unit 1)
-    (in_bom yes) (on_board yes) (dnp no) (fields_autoplaced)
-    (property "Reference" "H106" (at 134.62 176.9653 0)
+  (symbol (lib_id "Mechanical:MountingHole") (at 142.24 181.61 0) (unit 1)
+    (in_bom no) (on_board yes) (dnp no) (fields_autoplaced)
+    (property "Reference" "H106" (at 144.78 180.7753 0)
       (effects (font (size 1.27 1.27)) (justify left))
     )
-    (property "Value" "ToolingHole" (at 134.62 179.5022 0)
+    (property "Value" "ToolingHole" (at 144.78 183.3122 0)
       (effects (font (size 1.27 1.27)) (justify left))
     )
-    (property "Footprint" "JLC:JLC_toolinghole" (at 132.08 177.8 0)
+    (property "Footprint" "JLC:JLC_toolinghole" (at 142.24 181.61 0)
       (effects (font (size 1.27 1.27)) hide)
     )
-    (property "Datasheet" "~" (at 132.08 177.8 0)
+    (property "Datasheet" "~" (at 142.24 181.61 0)
       (effects (font (size 1.27 1.27)) hide)
     )
@@
   )
   (symbol (lib_id "Mechanical:MountingHole_Pad") (at 236.22 142.24 0) (unit 1)
-    (in_bom yes) (on_board yes) (dnp no) (fields_autoplaced)
+    (in_bom no) (on_board yes) (dnp no) (fields_autoplaced)
     (property "Reference" "H103" (at 238.76 140.1353 0)
       (effects (font (size 1.27 1.27)) (justify left))
@@
   )
   (symbol (lib_id "Mechanical:MountingHole_Pad") (at 215.9 142.24 0) (unit 1)
-    (in_bom yes) (on_board yes) (dnp no)
+    (in_bom no) (on_board yes) (dnp no)
     (property "Reference" "H102" (at 218.44 140.1353 0)
       (effects (font (size 1.27 1.27)) (justify left))
@@
   )
   (symbol (lib_id "Mechanical:MountingHole_Pad") (at 195.58 142.24 0) (unit 1)
-    (in_bom yes) (on_board yes) (dnp no) (fields_autoplaced)
+    (in_bom no) (on_board yes) (dnp no) (fields_autoplaced)
     (property "Reference" "H101" (at 198.12 140.1353 0)
       (effects (font (size 1.27 1.27)) (justify left))
@@
     )
   )
-  (symbol (lib_id "Mechanical:MountingHole") (at 111.76 177.8 270) (unit 1)
-    (in_bom yes) (on_board yes) (dnp no)
-    (property "Reference" "H105" (at 114.3 176.9653 90)
+  (symbol (lib_id "Mechanical:MountingHole") (at 121.92 181.61 270) (unit 1)
+    (in_bom no) (on_board yes) (dnp no)
+    (property "Reference" "H105" (at 124.46 180.7753 90)
       (effects (font (size 1.27 1.27)) (justify left))
     )
-    (property "Value" "ToolingHole" (at 114.3 179.5022 90)
+    (property "Value" "ToolingHole" (at 124.46 183.3122 90)
       (effects (font (size 1.27 1.27)) (justify left))
     )
-    (property "Footprint" "JLC:JLC_toolinghole" (at 111.76 177.8 0)
+    (property "Footprint" "JLC:JLC_toolinghole" (at 121.92 181.61 0)
       (effects (font (size 1.27 1.27)) hide)
     )
-    (property "Datasheet" "~" (at 111.76 177.8 0)
+    (property "Datasheet" "~" (at 121.92 181.61 0)
       (effects (font (size 1.27 1.27)) hide)
     )
