File: leds.kicad_sch (KiCad schematic)
At the start: 64 parts

Commit message: Change LCSC partnumbers for LEDS and NM for testpoints
Parts:
- D301, D302, D303, D304, D305, D306, D307, D308, D309, D310, D311, D312, D313, D314, D315, D316, D317, D318, D319, D320, D321, D322, D323, D324, D325: LCSC C2874885 -> C2920042
- TP301, TP302, TP303, TP304, TP305, TP306, TP307, TP308, TP309, TP310, TP311, TP312: LCSC C238122 -> (none)
Changed lines of the file:
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@@
       (effects (font (size 1.27 1.27)) (justify left top) hide)
     )
-    (property "LCSC" "C2874885" (id 4) (at 114.935 124.46 0)
+    (property "LCSC" "C2920042" (id 4) (at 114.935 124.46 0)
       (effects (font (size 1.27 1.27)) hide)
     )
@@
       (effects (font (size 1.27 1.27)) (justify left top) hide)
     )
-    (property "LCSC" "C2874885" (id 4) (at 92.075 154.94 0)
+    (property "LCSC" "C2920042" (id 4) (at 92.075 154.94 0)
       (effects (font (size 1.27 1.27)) hide)
     )
@@
       (effects (font (size 1.27 1.27)) hide)
     )
-    (property "LCSC" "C238122" (id 4) (at 33.02 185.42 0)
+    (property "LCSC" "" (id 4) (at 33.02 185.42 0)
       (effects (font (size 1.27 1.27)) hide)
     )
@@
       (effects (font (size 1.27 1.27)) (justify left top) hide)
     )
-    (property "LCSC" "C2874885" (id 4) (at 160.655 154.94 0)
+    (property "LCSC" "C2920042" (id 4) (at 160.655 154.94 0)
       (effects (font (size 1.27 1.27)) hide)
     )
@@
       (effects (font (size 1.27 1.27)) (justify left top) hide)
     )
-    (property "LCSC" "C2874885" (id 4) (at 92.075 63.5 0)
+    (property "LCSC" "C2920042" (id 4) (at 92.075 63.5 0)
       (effects (font (size 1.27 1.27)) hide)
     )
@@
       (effects (font (size 1.27 1.27)) (justify left top) hide)
     )
-    (property "LCSC" "C2874885" (id 4) (at 69.215 154.94 0)
+    (property "LCSC" "C2920042" (id 4) (at 69.215 154.94 0)
       (effects (font (size 1.27 1.27)) hide)
     )
@@
       (effects (font (size 1.27 1.27)) hide)
     )
-    (property "LCSC" "C238122" (id 4) (at 63.5 185.42 0)
+    (property "LCSC" "" (id 4) (at 63.5 185.42 0)
       (effects (font (size 1.27 1.27)) hide)
     )
@@
       (effects (font (size 1.27 1.27)) (justify left top) hide)
     )
-    (property "LCSC" "C2874885" (id 4) (at 69.215 63.5 0)
+    (property "LCSC" "C2920042" (id 4) (at 69.215 63.5 0)
       (effects (font (size 1.27 1.27)) hide)
     )
@@
       (effects (font (size 1.27 1.27)) (justify left top) hide)
     )
-    (property "LCSC" "C2874885" (id 4) (at 160.655 63.5 0)
+    (property "LCSC" "C2920042" (id 4) (at 160.655 63.5 0)
       (effects (font (size 1.27 1.27)) hide)
     )
@@
       (effects (font (size 1.27 1.27)) hide)
     )
-    (property "LCSC" "C238122" (id 4) (at 173.355 93.98 0)
+    (property "LCSC" "" (id 4) (at 173.355 93.98 0)
       (effects (font (size 1.27 1.27)) hide)
     )
@@
       (effects (font (size 1.27 1.27)) (justify left top) hide)
     )
-    (property "LCSC" "C2874885" (id 4) (at 114.935 33.02 0)
+    (property "LCSC" "C2920042" (id 4) (at 114.935 33.02 0)
       (effects (font (size 1.27 1.27)) hide)
     )
@@
       (effects (font (size 1.27 1.27)) (justify left top) hide)
     )
-    (property "LCSC" "C2874885" (id 4) (at 114.935 63.5 0)
+    (property "LCSC" "C2920042" (id 4) (at 114.935 63.5 0)
       (effects (font (size 1.27 1.27)) hide)
     )
@@
       (effects (font (size 1.27 1.27)) (justify left top) hide)
     )
-    (property "LCSC" "C2874885" (id 4) (at 160.655 124.46 0)
+    (property "LCSC" "C2920042" (id 4) (at 160.655 124.46 0)
       (effects (font (size 1.27 1.27)) hide)
     )
@@
       (effects (font (size 1.27 1.27)) (justify left top) hide)
     )
-    (property "LCSC" "C2874885" (id 4) (at 69.215 124.46 0)
+    (property "LCSC" "C2920042" (id 4) (at 69.215 124.46 0)
       (effects (font (size 1.27 1.27)) hide)
     )
@@
       (effects (font (size 1.27 1.27)) (justify left top) hide)
     )
-    (property "LCSC" "C2874885" (id 4) (at 137.795 93.98 0)
+    (property "LCSC" "C2920042" (id 4) (at 137.795 93.98 0)
       (effects (font (size 1.27 1.27)) hide)
     )
@@
       (effects (font (size 1.27 1.27)) hide)
     )
-    (property "LCSC" "C238122" (id 4) (at 43.18 33.02 0)
+    (property "LCSC" "" (id 4) (at 43.18 33.02 0)
       (effects (font (size 1.27 1.27)) hide)
     )
@@
       (effects (font (size 1.27 1.27)) (justify left top) hide)
     )
-    (property "LCSC" "C2874885" (id 4) (at 160.655 33.02 0)
+    (property "LCSC" "C2920042" (id 4) (at 160.655 33.02 0)
       (effects (font (size 1.27 1.27)) hide)
     )
@@
       (effects (font (size 1.27 1.27)) hide)
     )
-    (property "LCSC" "C238122" (id 4) (at 22.86 185.42 0)
+    (property "LCSC" "" (id 4) (at 22.86 185.42 0)
       (effects (font (size 1.27 1.27)) hide)
     )
@@
       (effects (font (size 1.27 1.27)) (justify left top) hide)
     )
-    (property "LCSC" "C2874885" (id 4) (at 114.935 154.94 0)
+    (property "LCSC" "C2920042" (id 4) (at 114.935 154.94 0)
       (effects (font (size 1.27 1.27)) hide)
     )
@@
       (effects (font (size 1.27 1.27)) (justify left top) hide)
     )
-    (property "LCSC" "C2874885" (id 4) (at 137.795 33.02 0)
+    (property "LCSC" "C2920042" (id 4) (at 137.795 33.02 0)
       (effects (font (size 1.27 1.27)) hide)
     )
@@
       (effects (font (size 1.27 1.27)) (justify left top) hide)
     )
-    (property "LCSC" "C2874885" (id 4) (at 69.215 93.98 0)
+    (property "LCSC" "C2920042" (id 4) (at 69.215 93.98 0)
       (effects (font (size 1.27 1.27)) hide)
     )
@@
       (effects (font (size 1.27 1.27)) (justify left top) hide)
     )
-    (property "LCSC" "C2874885" (id 4) (at 137.795 124.46 0)
+    (property "LCSC" "C2920042" (id 4) (at 137.795 124.46 0)
       (effects (font (size 1.27 1.27)) hide)
     )
@@
       (effects (font (size 1.27 1.27)) (justify left top) hide)
     )
-    (property "LCSC" "C2874885" (id 4) (at 69.215 33.02 0)
+    (property "LCSC" "C2920042" (id 4) (at 69.215 33.02 0)
       (effects (font (size 1.27 1.27)) hide)
     )
@@
       (effects (font (size 1.27 1.27)) (justify left top) hide)
     )
-    (property "LCSC" "C2874885" (id 4) (at 92.075 124.46 0)
+    (property "LCSC" "C2920042" (id 4) (at 92.075 124.46 0)
       (effects (font (size 1.27 1.27)) hide)
     )
@@
       (effects (font (size 1.27 1.27)) hide)
     )
-    (property "LCSC" "C238122" (id 4) (at 170.815 154.94 0)
+    (property "LCSC" "" (id 4) (at 170.815 154.94 0)
       (effects (font (size 1.27 1.27)) hide)
     )
@@
       (effects (font (size 1.27 1.27)) (justify left top) hide)
     )
-    (property "LCSC" "C2874885" (id 4) (at 92.075 93.98 0)
+    (property "LCSC" "C2920042" (id 4) (at 92.075 93.98 0)
       (effects (font (size 1.27 1.27)) hide)
     )
@@
       (effects (font (size 1.27 1.27)) (justify left top) hide)
     )
-    (property "LCSC" "C2874885" (id 4) (at 160.655 93.98 0)
+    (property "LCSC" "C2920042" (id 4) (at 160.655 93.98 0)
       (effects (font (size 1.27 1.27)) hide)
     )
@@
       (effects (font (size 1.27 1.27)) (justify left top) hide)
     )
-    (property "LCSC" "C2874885" (id 4) (at 92.075 33.02 0)
+    (property "LCSC" "C2920042" (id 4) (at 92.075 33.02 0)
       (effects (font (size 1.27 1.27)) hide)
     )
@@
       (effects (font (size 1.27 1.27)) (justify left top) hide)
     )
-    (property "LCSC" "C2874885" (id 4) (at 137.795 154.94 0)
+    (property "LCSC" "C2920042" (id 4) (at 137.795 154.94 0)
       (effects (font (size 1.27 1.27)) hide)
     )
@@
       (effects (font (size 1.27 1.27)) (justify left top) hide)
     )
-    (property "LCSC" "C2874885" (id 4) (at 114.935 93.98 0)
+    (property "LCSC" "C2920042" (id 4) (at 114.935 93.98 0)
       (effects (font (size 1.27 1.27)) hide)
     )
@@
       (effects (font (size 1.27 1.27)) (justify left top) hide)
     )
-    (property "LCSC" "C2874885" (id 4) (at 137.795 63.5 0)
+    (property "LCSC" "C2920042" (id 4) (at 137.795 63.5 0)
       (effects (font (size 1.27 1.27)) hide)
     )
@@
       (effects (font (size 1.27 1.27)) hide)
     )
-    (property "LCSC" "C238122" (id 4) (at 73.66 185.42 0)
+    (property "LCSC" "" (id 4) (at 73.66 185.42 0)
       (effects (font (size 1.27 1.27)) hide)
     )
@@
       (effects (font (size 1.27 1.27)) hide)
     )
-    (property "LCSC" "C238122" (id 4) (at 53.34 185.42 0)
+    (property "LCSC" "" (id 4) (at 53.34 185.42 0)
       (effects (font (size 1.27 1.27)) hide)
     )
@@
       (effects (font (size 1.27 1.27)) hide)
     )
-    (property "LCSC" "C238122" (id 4) (at 43.18 185.42 0)
+    (property "LCSC" "" (id 4) (at 43.18 185.42 0)
       (effects (font (size 1.27 1.27)) hide)
     )
@@
       (effects (font (size 1.27 1.27)) hide)
     )
-    (property "LCSC" "C238122" (id 4) (at 173.355 33.02 0)
+    (property "LCSC" "" (id 4) (at 173.355 33.02 0)
       (effects (font (size 1.27 1.27)) hide)
     )
@@
       (effects (font (size 1.27 1.27)) hide)
     )
-    (property "LCSC" "C238122" (id 4) (at 56.515 124.46 0)
+    (property "LCSC" "" (id 4) (at 56.515 124.46 0)
       (effects (font (size 1.27 1.27)) hide)
     )
@@
       (effects (font (size 1.27 1.27)) hide)
     )
-    (property "LCSC" "C238122" (id 4) (at 56.515 63.5 0)
-      (effects (font (size 1.27 1.27)) hide)
-    )
+    (property "LCSC" "" (id 4) (at 56.515 63.5 0)
+      (effects (font (size 1.27 1.27)) hide)
+    )
